Commit message: Finalize joint limits

File: description/robot.urdf (robot description, URDF)
Before this commit: robot str1ker, 6 links, 5 joints
Joints:
- joint elbow: limit lower=-2.2 upper=0.7 effort=155.68776 velocity=1.0 -> lower=-1.8 upper=-0.9 effort=155.68776 velocity=1.0
- joint shoulder: limit lower=-2.2 upper=0.7 effort=24 velocity=1.0 -> lower=0 upper=0.785398 effort=24 velocity=1.0; origin xyz=0 0.0127 0.108839 rpy=0 0 0 -> xyz=0 -0.0127 0.108839 rpy=0 0 0
- joint wrist: limit lower=-2.2 upper=0.7 effort=88.96443 velocity=1.0 -> lower=1.2 upper=1.3 effort=88.96443 velocity=1.0; origin xyz=0 0.4173 0 rpy=0 0 0 -> xyz=0 0.48059393086 0 rpy=0 0 0

Commit message: Add drumstick collision geometry

File: description/robot.urdf (robot description, URDF)
Before this commit: robot str1ker, 6 links, 5 joints
Links:
- link drumstick_link: geometry collision mesh filename=package://str1ker/description/models/DrumstickBoundingBox.s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; visual mesh filename=package://str1ker/description/models/Drumstick.stl

Commit message: Fill in physical descriptions

File: description/robot.urdf (robot description, URDF)
Before this commit: robot str1ker, 6 links, 5 joints
Links:
- link base_link: mass 35.336455 -> None
- link drumstick_link: mass 0.336455 -> 0.091
- link forearm_link: mass 35.336455 -> 0.703
- link shoulder_link: mass 35.336455 -> 0.36378108
- link upperarm_link: mass 35.336455 -> 1.139
Joints:
- joint elbow: limit lower=-1.8 upper=-0.9 effort=155.68776 velocity=1.0 -> lower=-1.8 upper=-0.9 effort=100 velocity=1.0
- joint shoulder: limit lower=0 upper=0.785398 effort=24 velocity=1.0 -> lower=0 upper=0.785398 effort=100 velocity=1.0
- joint wrist: limit lower=1.2 upper=1.3 effort=88.96443 velocity=1.0 -> lower=1.2 upper=1.3 effort=100 velocity=1.0

Commit message: Fix arm turning

File: description/robot.urdf (robot description, URDF)
Before this commit: robot str1ker, 6 links, 5 joints
Joints:
- removed joint arm_mount
- added joint mount: type revolute, parent base_link, child shoulder_link, origin xyz=0 0 0 rpy=0 0 0, axis 0 0 1, limit lower=-1.4929 upper=1.4929 effort=100 velocity=1.0

Commit message: Add actuator links and joints

File: description/robot.urdf (robot description, URDF)
Before this commit: robot str1ker, 6 links, 5 joints
Links:
- added link forearm_actuator_body_link, mass 0.199; collision mesh filename=package://str1ker/description/models/TODO.stl; visual mesh filename=package://str1ker/description/models/ForearmActuatorBody.stl
- added link forearm_actuator_shaft_link, mass 0.113; collision mesh filename=package://str1ker/description/models/TODO.stl; visual mesh filename=package://str1ker/description/models/ForearmActuatorShaft.s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
- added link upperarm_actuator_body_link, mass 0.796; collision mesh filename=package://str1ker/description/models/TODO.stl; visual mesh filename=package://str1ker/description/models/UpperArmActuatorBody.s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
- added link upperarm_actuator_shaft_link, mass 0.070; collision mesh filename=package://str1ker/description/models/TODO.stl; visual mesh filename=package://str1ker/description/models/UpperArmActuatorShaft.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
Joints:
- added joint forearm_actuator_base: type revolute , parent upperarm_link, child forearm_actuator_body_link, origin xyz=0 0.130 -0.034 rpy=0 0 0, axis 1 0 0, limit lower=0 upper=2 effort=100 velocity=1.0
- added joint forearm_actuator_shaft: type prismatic, parent forearm_actuator_body_link, child forearm_actuator_shaft_link, origin xyz=0 0 0.135 rpy=0 0 0, axis 0 0 1, limit lower=0 upper=2 effort=100 velocity=1.0
- added joint forearm_actuator_shaft_end: type revolute , parent forearm_actuator_shaft_link, child forearm_link, origin xyz=0 0 0.137 rpy=0 0 0, axis 1 0 0, limit lower=0 upper=2 effort=100 velocity=1.0
- added joint shoulder_actuator_base: type revolute , parent shoulder_link, child upperarm_actuator_body_link, origin xyz=0 0.101 -0.057 rpy=0 0 0, axis 1 0 0, limit lower=0 upper=2 effort=100 velocity=1.0
- added joint shoulder_actuator_shaft: type prismatic, parent upperarm_actuator_body_link, child upperarm_actuator_shaft_link, origin xyz=0 -0.002 0.184 rpy=0 0 0, axis 0 0 1, limit lower=0 upper=2 effort=100 velocity=1.0
- added joint shoulder_actuator_shaft_end: type revolute , parent upperarm_actuator_shaft_link, child upperarm_link, origin xyz=0 0 0.083 rpy=0 0 0, axis 1 0 0, limit lower=0 upper=2 effort=100 velocity=1.0

Commit message: Update actuator chains

File: description/robot.urdf (robot description, URDF)
Before this commit: robot str1ker, 10 links, 11 joints
Links:
- added link forearm_actuator_target_link; visual sphere radius=0.005
- added link upperarm_actuator_target_link; visual sphere radius=0.005
Joints:
- removed joint shoulder_actuator_base
- removed joint shoulder_actuator_shaft
- removed joint shoulder_actuator_shaft_end
- added joint forearm_actuator_target: type revolute, parent forearm_link, child forearm_actuator_target_link, origin xyz=0 0.069 -0.06 rpy=0 0 0, axis 1 0 0, limit lower=-2 upper=2 effort=100 velocity=1.0
- added joint upperarm_actuator_base: type revolute, parent shoulder_link, child upperarm_actuator_body_link, origin xyz=0 0.101 -0.057 rpy=0 0 0, axis 1 0 0, limit lower=-1 upper=0 effort=100 velocity=1.0
- added joint upperarm_actuator_shaft: type prismatic, parent upperarm_actuator_body_link, child upperarm_actuator_shaft_link, origin xyz=0 0.002 0.184 rpy=0 0 0, axis 0 0 1, limit lower=-2 upper=0 effort=100 velocity=1.0
- added joint upperarm_actuator_shaft_end: type revolute, parent upperarm_actuator_shaft_link, child upperarm_actuator_target_link, origin xyz=0 0 0.083 rpy=0 0 0, axis 1 0 0, limit lower=-2 upper=2 effort=100 velocity=1.0
- added joint upperarm_actuator_target: type revolute, parent upperarm_link, child upperarm_actuator_target_link, origin xyz=0 0.11 -0.054 rpy=0 0 0, axis 1 0 0, limit lower=-2 upper=2 effort=100 velocity=1.0
- joint forearm_actuator_base: limit lower=0 upper=2 effort=100 velocity=1.0 -> lower=-1 upper=0 effort=100 velocity=1.0; type revolute  -> revolute
- joint forearm_actuator_shaft: axis 0 0 1 -> 0 1 0; limit lower=0 upper=2 effort=100 velocity=1.0 -> lower=-1 upper=0 effort=100 velocity=1.0; origin xyz=0 0 0.135 rpy=0 0 0 -> xyz=0 0.135 0 rpy=0 0 0
- joint forearm_actuator_shaft_end: child forearm_link -> forearm_actuator_target_link; type revolute  -> revolute
- joint shoulder: limit lower=0 upper=0.785398 effort=100 velocity=1.0 -> lower=0.75 upper=1.0 effort=100 velocity=1.0

Commit message: Round of cleaning up urdf

File: description/robot.urdf (robot description, URDF)
Before this commit: robot str1ker, 12 links, 13 joints
Links:
- removed link forearm_actuator_shaft_link
- removed link forearm_actuator_target_link
- removed link upperarm_actuator_shaft_link
- removed link upperarm_actuator_target_link
- added link forearm_actuator_link, mass 0.113; collision mesh filename=package://str1ker/description/models/TODO.stl; visual mesh filename=package://str1ker/description/models/ForearmActuatorShaft.s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
- added link upperarm_actuator_link, mass 0.070; collision mesh filename=package://str1ker/description/models/TODO.stl; visual mesh filename=package://str1ker/description/models/UpperArmActuatorShaft.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
Joints:
- removed joint forearm_actuator_base
- removed joint forearm_actuator_shaft
- removed joint forearm_actuator_shaft_end
- removed joint forearm_actuator_target
- removed joint upperarm_actuator_base
- removed joint upperarm_actuator_shaft
- removed joint upperarm_actuator_shaft_end
- removed joint upperarm_actuator_target
- added joint forearm_actuator: type prismatic, parent forearm_actuator_body_link, child forearm_actuator_link, origin xyz=0 0.135 0 rpy=0 0 0, axis 0 1 0, limit lower=-0.0508 upper=0 effort=100 velocity=1.0
- added joint forearm_actuator_mount: type revolute, parent upperarm_link, child forearm_actuator_body_link, origin xyz=0 0.130 -0.034 rpy=0 0 0, axis 1 0 0, limit lower=-0.1 upper=0.1 effort=100 velocity=1.0
- added joint upperarm_actuator: type prismatic, parent upperarm_actuator_body_link, child upperarm_actuator_link, origin xyz=0 0.002 0.184 rpy=0 0 0, axis 0 0 1, limit lower=-0.0508 upper=0 effort=100 velocity=1.0
- added joint upperarm_actuator_mount: type revolute, parent shoulder_link, child upperarm_actuator_body_link, origin xyz=0 0.101045 -0.0504975 rpy=0 0 0, axis 1 0 0, limit lower=-0.2 upper=-0.0500 effort=100 velocity=1.0
- joint elbow: limit lower=-1.8 upper=-0.9 effort=100 velocity=1.0 -> lower=-1.9 upper=-0.9243 effort=100 velocity=1.0
- joint mount: origin xyz=0 0 0 rpy=0 0 0 -> xyz=0 0 0.0055 rpy=0 0 0
- joint shoulder: limit lower=0.75 upper=1.0 effort=100 velocity=1.0 -> lower=0.43 upper=0.6361 effort=100 velocity=1.0; origin xyz=0 -0.0127 0.108839 rpy=0 0 0 -> xyz=0 -0.013 0.11518 rpy=0 0 0
- joint wrist: limit lower=1.2 upper=1.3 effort=100 velocity=1.0 -> lower=1 upper=1.05 effort=100 velocity=1.0

Commit message: More cleaning on urdf

File: description/robot.urdf (robot description, URDF)
Before this commit: robot str1ker, 10 links, 9 joints
Links:
- removed link forearm_actuator_link
- removed link upperarm_actuator_link
- added link forearm_actuator_shaft_link, mass 0.113; collision mesh filename=package://str1ker/description/models/TODO.stl; visual mesh filename=package://str1ker/description/models/ForearmActuatorShaft.s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
- added link upperarm_actuator_shaft_link, mass 0.070; collision mesh filename=package://str1ker/description/models/TODO.stl; visual mesh filename=package://str1ker/description/models/UpperArmActuatorShaft.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
Joints:
- joint forearm_actuator: child forearm_actuator_link -> forearm_actuator_shaft_link
- joint forearm_actuator_mount: limit lower=-0.1 upper=0.1 effort=100 velocity=1.0 -> lower=-0.15 upper=0.0277 effort=100 velocity=1.0
- joint mount: origin xyz=0 0 0.0055 rpy=0 0 0 -> xyz=0 0 0 rpy=0 0 0
- joint shoulder: limit lower=0.43 upper=0.6361 effort=100 velocity=1.0 -> lower=0.4853 upper=0.6361 effort=100 velocity=1.0
- joint upperarm_actuator: child upperarm_actuator_link -> upperarm_actuator_shaft_link; origin xyz=0 0.002 0.184 rpy=0 0 0 -> xyz=0 -0.002 0.159 rpy=0 0 0
- joint upperarm_actuator_mount: limit lower=-0.2 upper=-0.0500 effort=100 velocity=1.0 -> lower=-0.2 upper=0.1 effort=100 velocity=1.0

Commit message: Wrist limit

File: description/robot.urdf (robot description, URDF)
Before this commit: robot str1ker, 10 links, 9 joints
Joints:
- joint wrist: limit lower=1 upper=1.05 effort=100 velocity=1.0 -> lower=2.55 upper=2.6 effort=100 velocity=1.0

Commit message: Update collision stls

File: description/robot.urdf (robot description, URDF)
Before this commit: robot str1ker, 10 links, 9 joints
Links:
- link forearm_actuator_body_link: geometry collision mesh filename=package://str1ker/description/models/ForearmActuatorBodyBou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; visual mesh filename=package://str1ker/description/models/ForearmActuatorBody.stl
- link forearm_actuator_shaft_link: geometry collision mesh filename=package://str1ker/description/models/ForearmActuatorShaftBo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; visual mesh filename=package://str1ker/description/models/ForearmActuatorShaft.s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
- link upperarm_actuator_body_link: geometry collision mesh filename=package://str1ker/description/models/UpperArmActuatorBodyBo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; visual mesh filename=package://str1ker/description/models/UpperArmActuatorBody.s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
- link upperarm_actuator_shaft_link: geometry collision mesh filename=package://str1ker/description/models/UpperArmActuatorShaftB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; visual mesh filename=package://str1ker/description/models/UpperArmActuatorShaft.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
Joints:
- joint forearm_actuator: origin xyz=0 0.135 0 rpy=0 0 0 -> xyz=0 0.210 0 rpy=0 0 0

Commit message: Fix wrist limit

File: description/robot.urdf (robot description, URDF)
Before this commit: robot str1ker, 10 links, 9 joints
Joints:
- joint wrist: limit lower=2.55 upper=2.6 effort=100 velocity=1.0 -> lower=0.7 upper=0.8 effort=100 velocity=1.0

Commit message: More precise upper arm actuator limit

File: description/robot.urdf (robot description, URDF)
Before this commit: robot str1ker, 10 links, 9 joints
Joints:
- joint upperarm_actuator: limit lower=-0.0508 upper=0 effort=100 velocity=1.0 -> lower=-0.0474 upper=0 effort=100 velocity=1.0

Commit message: Upper arm actuator mount rotation mimics shaft

File: description/robot.urdf (robot description, URDF)
Before this commit: robot str1ker, 10 links, 9 joints
Joints:
- joint upperarm_actuator_mount: limit lower=-0.2 upper=0.1 effort=100 velocity=1.0 -> lower=-0.1 upper=0 effort=100 velocity=1.0; mimic (none) -> joint=upperarm_actuator multiplier=0.25 offset=-0.05

Commit message: Best guess on limits and mimics

File: description/robot.urdf (robot description, URDF)
Before this commit: robot str1ker, 10 links, 9 joints
Joints:
- joint elbow: limit lower=-1.9 upper=-0.9243 effort=100 velocity=1.0 -> lower=-1.8762289 upper=-0.89528 effort=100 velocity=1.0; mimic (none) -> joint=forearm_actuator multiplier=19.311023622 offset=-0.8952
- joint forearm_actuator_mount: mimic (none) -> joint=forearm_actuator multiplier=-2.179133858 offset=-0.15
- joint shoulder: limit lower=0.4853 upper=0.6361 effort=100 velocity=1.0 -> lower=0.2879793 upper=0.6544985 effort=100 velocity=1.0; mimic (none) -> joint=upperarm_actuator multiplier=7.214944882 offset=0.6544985
- joint upperarm_actuator: limit lower=-0.0474 upper=0 effort=100 velocity=1.0 -> lower=-0.0508 upper=0 effort=100 velocity=1.0

Commit message: Shorten upper arm actuator body

File: description/robot.urdf (robot description, URDF)
Before this commit: robot str1ker, 10 links, 9 joints
Joints:
- joint upperarm_actuator: origin xyz=0 -0.002 0.159 rpy=0 0 0 -> xyz=0 -0.002 0.139 rpy=0 0 0

Commit message: Lengthen forearm actuator

File: description/robot.urdf (robot description, URDF)
Before this commit: robot str1ker, 10 links, 9 joints
Joints:
- joint forearm_actuator: origin xyz=0 0.210 0 rpy=0 0 0 -> xyz=0 0.225 0 rpy=0 0 0

Commit message: Update limits

File: description/robot.urdf (robot description, URDF)
Before this commit: robot str1ker, 10 links, 9 joints
Joints:
- joint elbow: limit lower=-1.8762289 upper=-0.89528 effort=100 velocity=1.0 -> lower=-1.590787 upper=-0.829031 effort=100 velocity=1.0; mimic joint=forearm_actuator multiplier=19.311023622 offset=-0.8952 -> joint=forearm_actuator multiplier=14.99519685 offset=-0.829031
- joint forearm_actuator_mount: limit lower=-0.15 upper=0.0277 effort=100 velocity=1.0 -> lower=-0.146607 upper=-0.118682 effort=100 velocity=1.0; mimic joint=forearm_actuator multiplier=-2.179133858 offset=-0.15 -> joint=forearm_actuator multiplier=-0.549606299 offset=-0.146602
- joint shoulder: limit lower=0.2879793 upper=0.6544985 effort=100 velocity=1.0 -> lower=0.303687 upper=0.691150 effort=100 velocity=1.0; mimic joint=upperarm_actuator multiplier=7.214944882 offset=0.6544985 -> joint=upperarm_actuator multiplier=7.627224409 offset=0.69115
- joint upperarm_actuator_mount: mimic joint=upperarm_actuator multiplier=0.25 offset=-0.05 -> joint=upperarm_actuator multiplier=0.618425197 offset=-0.05

Commit message: Tune upper arm actuator sim

File: description/robot.urdf (robot description, URDF)
Before this commit: robot str1ker, 10 links, 9 joints
Joints:
- joint upperarm_actuator: limit lower=-0.0508 upper=0 effort=100 velocity=1.0 -> lower=-0.0508 upper=-0.0005 effort=100 velocity=1.0
- joint upperarm_actuator_mount: mimic joint=upperarm_actuator multiplier=0.618425197 offset=-0.05 -> joint=upperarm_actuator multiplier=0.7 offset=-0.04

Commit message: Actuator notes

File: description/robot.urdf (robot description, URDF)
Before this commit: robot str1ker, 10 links, 9 joints
Joints:
- joint forearm_actuator: limit lower=-0.0508 upper=0 effort=100 velocity=1.0 -> lower=-0.0508 upper=0 effort=100 velocity=0.0109982
- joint upperarm_actuator: limit lower=-0.0508 upper=-0.0005 effort=100 velocity=1.0 -> lower=-0.0508 upper=-0.0005 effort=100 velocity=0.0508

Commit message: Revert "Lengthen forearm actuator"
This reverts commit 52cb549178ae56ad37ba80106483dcd69fc9dd6b.

File: description/robot.urdf (robot description, URDF)
Before this commit: robot str1ker, 10 links, 9 joints
Joints:
- joint forearm_actuator: origin xyz=0 0.225 0 rpy=0 0 0 -> xyz=0 0.210 0 rpy=0 0 0

Commit message: Revert "Shorten upper arm actuator body"
This reverts commit a84f4c9be8dbbe7efa7a3a994118b4b1107c95e8.

File: description/robot.urdf (robot description, URDF)
Before this commit: robot str1ker, 10 links, 9 joints
Joints:
- joint upperarm_actuator: origin xyz=0 -0.002 0.139 rpy=0 0 0 -> xyz=0 -0.002 0.159 rpy=0 0 0

Commit message: Shorten upper arm actuator to measured dims

File: description/robot.urdf (robot description, URDF)
Before this commit: robot str1ker, 10 links, 9 joints
Joints:
- joint upperarm_actuator: origin xyz=0 -0.002 0.159 rpy=0 0 0 -> xyz=0 -0.002 0.153 rpy=0 0 0

Commit message: Increase upper arm actuator limit todo

File: description/robot.urdf (robot description, URDF)
Before this commit: robot str1ker, 10 links, 9 joints
Joints:
- joint upperarm_actuator: limit lower=-0.0508 upper=-0.0005 effort=100 velocity=0.0508 -> lower=-0.054 upper=-0.0005 effort=100 velocity=0.0508

Commit message: Update shoulder mimic based on upper arm actuator change

File: description/robot.urdf (robot description, URDF)
Before this commit: robot str1ker, 10 links, 9 joints
Joints:
- joint shoulder: mimic joint=upperarm_actuator multiplier=7.627224409 offset=0.69115 -> joint=upperarm_actuator multiplier=7.242299065 offset=0.69477115

Commit message: Update elbow and shoulder limits from photo ref

File: description/robot.urdf (robot description, URDF)
Before this commit: robot str1ker, 10 links, 9 joints
Joints:
- joint elbow: limit lower=-1.590787 upper=-0.829031 effort=100 velocity=1.0 -> lower=-1.93302196 upper=-1.123992 effort=100 velocity=1.0
- joint shoulder: limit lower=0.303687 upper=0.691150 effort=100 velocity=1.0 -> lower=0.2391101 upper=0.6230825 effort=100 velocity=1.0

Commit message: Update elbow and shoulder mimics based on new limits

File: description/robot.urdf (robot description, URDF)
Before this commit: robot str1ker, 10 links, 9 joints
Joints:
- joint elbow: mimic joint=forearm_actuator multiplier=14.99519685 offset=-0.829031 -> joint=forearm_actuator multiplier=15.925786614 offset=-1.123992
- joint shoulder: mimic joint=upperarm_actuator multiplier=7.242299065 offset=0.69477115 -> joint=upperarm_actuator multiplier=2.611299773 offset=0.380120288

Commit message: Update upper arm actuator rotation

File: description/robot.urdf (robot description, URDF)
Before this commit: robot str1ker, 10 links, 9 joints
Joints:
- joint forearm_actuator_mount: mimic joint=forearm_actuator multiplier=-0.549606299 offset=-0.146602 -> joint=forearm_actuator multiplier=-2.5 offset=-0.146602
- joint shoulder: mimic joint=upperarm_actuator multiplier=2.611299773 offset=0.380120288 -> joint=upperarm_actuator multiplier=7.177054206 offset=0.626671027

Commit message: Update limits and transmissions again

File: description/robot.urdf (robot description, URDF)
Before this commit: robot str1ker, 10 links, 9 joints
Links:
- link upperarm_actuator_body_link: mass 0.796 -> 0.952544
Joints:
- joint shoulder: limit lower=0.2391101 upper=0.6230825 effort=100 velocity=1.0 -> lower=0.404676 upper=0.813453 effort=100 velocity=1.0; mimic joint=upperarm_actuator multiplier=7.177054206 offset=0.626671027 -> joint=upperarm_actuator multiplier=7.640691589 offset=0.817273346
- joint upperarm_actuator_mount: limit lower=-0.1 upper=0 effort=100 velocity=1.0 -> lower=-0.1 upper=0.1 effort=100 velocity=1.0; mimic joint=upperarm_actuator multiplier=0.7 offset=-0.04 -> joint=upperarm_actuator multiplier=0.9 offset=-0.01

Commit message: Add forearm connector link

File: description/robot.urdf (robot description, URDF)
Before this commit: robot str1ker, 10 links, 9 joints
Links:
- added link forearm_actuator_connector_link, mass 0.013; visual mesh filename=package://str1ker/description/models/ForearmActuatorConnect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

Commit message: Add forearm connector joint

File: description/robot.urdf (robot description, URDF)
Before this commit: robot str1ker, 11 links, 9 joints
Joints:
- added joint forearm_actuator_connector: type revolute, parent forearm_link, origin xyz=0 0.0605718 0.004 rpy=0 0 0, axis 1 0 0, limit lower=-1 upper=1 effort=100 velocity=1.0

Commit message: Test connector link

File: description/robot.urdf (robot description, URDF)
Before this commit: robot str1ker, 11 links, 10 joints
Joints:
- joint forearm_actuator_connector: child (none) -> forearm_actuator_connector_link; limit lower=-1 upper=1 effort=100 velocity=1.0 -> lower=1.5137 upper=1.5444 effort=100 velocity=1.0; mimic (none) -> joint=forearm_actuator multiplier=0.604330709 offset=1.5444

Commit message: Export forearm actuator connector bounding box

File: description/robot.urdf (robot description, URDF)
Before this commit: robot str1ker, 11 links, 10 joints
Links:
- link forearm_actuator_connector_link: geometry collision mesh filename=package://str1ker/description/models/ForearmActuatorConnect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; visual mesh filename=package://str1ker/description/models/ForearmActuatorConnect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

Commit message: Initial urdf for arm solenoid

File: description/robot.urdf (robot description, URDF)
Before this commit: robot str1ker, 11 links, 10 joints
Links:
- added link solenoid_mount_link; visual mesh filename=package://str1ker/description/models/ArmSolenoid.stl
- added link solenoid_shaft_link; visual mesh filename=package://str1ker/description/models/ArmSolenoidShaft.stl
Joints:
- added joint solenoid: type prismatic, parent solenoid_mount_link, child solenoid_shaft_link, origin xyz=-0.017 -0.013 0.095 rpy=0 0 0, axis 0 0 1, limit lower=-1 upper=1 effort=100 velocity=1.0
- added joint solenoid_mount: type revolute, parent forearm_link, child solenoid_mount_link, origin xyz=0.013 0.355 -0.031 rpy=0 0 0, axis 1 0 0, limit lower=1.25 upper=1.9 effort=100 velocity=1.0

Commit message: Solenoid limits

File: description/robot.urdf (robot description, URDF)
Before this commit: robot str1ker, 13 links, 12 joints
Joints:
- joint solenoid: limit lower=-1 upper=1 effort=100 velocity=1.0 -> lower=-0.0019 upper=0.001 effort=100 velocity=1.0; origin xyz=-0.017 -0.013 0.095 rpy=0 0 0 -> xyz=0 0 0 rpy=0 0 0

Commit message: Wrist limits

File: description/robot.urdf (robot description, URDF)
Before this commit: robot str1ker, 13 links, 12 joints
Joints:
- joint wrist: limit lower=0.7 upper=0.8 effort=100 velocity=1.0 -> lower=1.0 upper=1.02 effort=100 velocity=1.0

Commit message: Tune wrist solenoid

File: description/robot.urdf (robot description, URDF)
Before this commit: robot str1ker, 13 links, 12 joints
Joints:
- joint wrist: mimic (none) -> joint=solenoid multiplier=-6.8966 offset=1.0069
