Commit message: Add solenoid collision urdf

File: description/robot.urdf (robot description, URDF)
Before this commit: robot str1ker, 13 links, 12 joints
Links:
- link solenoid_mount_link: geometry collision mesh filename=package://str1ker/description/models/ArmSolenoidBoundingBox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; visual mesh filename=package://str1ker/description/models/ArmSolenoid.stl
- link solenoid_shaft_link: geometry collision mesh filename=package://str1ker/description/models/ArmSolenoidShaftBoundi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; visual mesh filename=package://str1ker/description/models/ArmSolenoidShaft.stl

Commit message: Fix wrist x offset

File: description/robot.urdf (robot description, URDF)
Before this commit: robot str1ker, 13 links, 12 joints
Joints:
- joint wrist: origin xyz=0 0.48059393086 0 rpy=0 0 0 -> xyz=-0.009 0.48059393086 0 rpy=0 0 0

Commit message: Let moveit update urdf

File: description/robot.urdf (robot description, URDF)
Before this commit: robot str1ker, 13 links, 12 joints
Links:
- link solenoid_mount_link: mass None -> 0.1
- link solenoid_shaft_link: mass None -> 0.1

Commit message: Implement servo node

File: description/robot.urdf (robot description, URDF)
Before this commit: robot str1ker, 13 links, 12 joints
Joints:
- joint elbow: mimic joint=forearm_actuator multiplier=15.925786614 offset=-1.123992 -> (none)
- joint shoulder: mimic joint=upperarm_actuator multiplier=7.640691589 offset=0.817273346 -> (none)
- joint wrist: mimic joint=solenoid multiplier=-6.8966 offset=1.0069 -> (none)

Commit message: Use new initialization method instead of deprecated

File: description/robot.urdf (robot description, URDF)
Before this commit: robot str1ker, 12 links, 11 joints
Links:
- link base_link: mass 0.1 -> None

Commit message: Effector link with one planning group

File: description/robot.urdf (robot description, URDF)
Before this commit: robot str1ker, 12 links, 11 joints
Links:
- added link effector_link, mass 0.001; collision sphere radius=0.02; visual sphere radius=0.02
Joints:
- added joint effector: type fixed, parent forearm_link, child effector_link, origin xyz=-0.02 0.66 0.25 rpy=0 0 0

Commit message: Hide effector

File: description/robot.urdf (robot description, URDF)
Before this commit: robot str1ker, 13 links, 12 joints
Links:
- link effector_link: geometry collision sphere radius=0.02

Commit message: Fix build errors

File: description/robot.urdf (robot description, URDF)
Before this commit: robot str1ker, 13 links, 12 joints
Links:
- removed link effector_link
Joints:
- removed joint effector
- removed joint mount
- added joint base: type revolute, parent base_link, child shoulder_link, origin xyz=0 0 0 rpy=0 0 0, axis 0 0 1, limit lower=-1.4929 upper=1.4929 effort=100 velocity=1.0

Commit message: First pass fixing urdf, need stl export again

File: description/robot.urdf (robot description, URDF)
Before this commit: robot str1ker, 12 links, 11 joints
Links:
- added link tip_link; collision sphere radius=0.01; visual sphere radius=0.01
Joints:
- added joint tip: type fixed, parent drumstick_link, child tip_link, origin xyz=0.305 0.0 0.0 rpy=0 0 0
- joint base: axis 0 0 1 -> 0 1 0; origin xyz=0 0 0 rpy=0 0 0 -> xyz=0 0 0 rpy=1.5708 0 0
- joint elbow: axis 1 0 0 -> 0 0 1; origin xyz=0 0.4173 0 rpy=0 0 0 -> xyz=0.4173 0 0 rpy=0 0 0
- joint forearm_actuator: axis 0 1 0 -> 0 0 1
- joint forearm_actuator_connector: axis 1 0 0 -> 0 0 1
- joint forearm_actuator_mount: axis 1 0 0 -> 0 0 1
- joint shoulder: axis 1 0 0 -> 0 0 1; origin xyz=0 -0.013 0.11518 rpy=0 0 0 -> xyz=-0.013 0.11518 0.0 rpy=0 0 0
- joint solenoid_mount: axis 1 0 0 -> 0 0 1
- joint upperarm_actuator_mount: axis 1 0 0 -> 0 0 1
- joint wrist: axis 1 0 0 -> 0 0 1; origin xyz=-0.009 0.48059393086 0 rpy=0 0 0 -> xyz=0.48059393086 0 -0.023 rpy=0 0 0

Commit message: Fix joints after re-orientation

File: description/robot.urdf (robot description, URDF)
Before this commit: robot str1ker, 13 links, 12 joints
Joints:
- joint forearm_actuator: origin xyz=0 0.210 0 rpy=0 0 0 -> xyz=0.210 0 0 rpy=0 0 0
- joint forearm_actuator_connector: origin xyz=0 0.0605718 0.004 rpy=0 0 0 -> xyz=0.0605718 0.004 0 rpy=0 0 0
- joint forearm_actuator_mount: origin xyz=0 0.130 -0.034 rpy=0 0 0 -> xyz=0.130 -0.034 0 rpy=0 0 0
- joint solenoid_mount: origin xyz=0.013 0.355 -0.031 rpy=0 0 0 -> xyz=0.355 -0.031 0.013 rpy=0 0 0
- joint upperarm_actuator: origin xyz=0 -0.002 0.153 rpy=0 0 0 -> xyz=0.153 -0.002 0 rpy=0 0 0
- joint upperarm_actuator_mount: origin xyz=0 0.101045 -0.0504975 rpy=0 0 0 -> xyz=0.101045 -0.0504975 0 rpy=0 0 0

Commit message: Fix prismatic axis

File: description/robot.urdf (robot description, URDF)
Before this commit: robot str1ker, 13 links, 12 joints
Joints:
- joint forearm_actuator: axis 0 0 1 -> 1 0 0
- joint upperarm_actuator: axis 0 0 1 -> 1 0 0

Commit message: Adjust mimic and secondary joints

File: description/robot.urdf (robot description, URDF)
Before this commit: robot str1ker, 13 links, 12 joints
Joints:
- joint solenoid_mount: limit lower=1.25 upper=1.9 effort=100 velocity=1.0 -> lower=-0.09 upper=-0.09 effort=100 velocity=1.0
- joint upperarm_actuator_mount: limit lower=-0.1 upper=0.1 effort=100 velocity=1.0 -> lower=-1 upper=1 effort=100 velocity=1.0; mimic joint=upperarm_actuator multiplier=0.9 offset=-0.01 -> joint=upperarm_actuator multiplier=0.9 offset=1.560796327
- joint wrist: limit lower=1.0 upper=1.02 effort=100 velocity=1.0 -> lower=0.959931 upper=0.959931 effort=100 velocity=1.0

Commit message: Fix mimic limits

File: description/robot.urdf (robot description, URDF)
Before this commit: robot str1ker, 13 links, 12 joints
Joints:
- joint forearm_actuator_mount: limit lower=-0.146607 upper=-0.118682 effort=100 velocity=1.0 -> lower=-0.06 upper=0 effort=100 velocity=1.0
- joint upperarm_actuator_mount: limit lower=-1 upper=1 effort=100 velocity=1.0 -> lower=1.93 upper=2.293 effort=100 velocity=1.0

Commit message: Update inertia for base link

File: description/robot.urdf (robot description, URDF)
Before this commit: robot str1ker, 13 links, 12 joints
Links:
- link base_link: mass None -> 0.528

Commit message: Troubleshooting gazebo launch

File: description/robot.urdf (robot description, URDF)
Before this commit: robot str1ker, 13 links, 12 joints
Links:
- removed link forearm_actuator_body_link
- removed link forearm_actuator_connector_link
- removed link forearm_actuator_shaft_link
- removed link solenoid_mount_link
- removed link solenoid_shaft_link
- removed link upperarm_actuator_body_link
- removed link upperarm_actuator_shaft_link
- added link world
Joints:
- removed joint forearm_actuator
- removed joint forearm_actuator_connector
- removed joint forearm_actuator_mount
- removed joint solenoid
- removed joint solenoid_mount
- removed joint upperarm_actuator
- removed joint upperarm_actuator_mount
- added joint fixed: type fixed, parent world, child base_link, origin xyz=0 0 0.06 rpy=0 0 0
- joint base: origin xyz=0 0 0 rpy=1.5708 0 0 -> xyz=0 0 0.069 rpy=1.5708 0 0
- joint wrist: mimic joint=solenoid multiplier=-6.8966 offset=1.0069 -> (none)

Commit message: Turn off gravity and pause on startup

File: description/robot.urdf (robot description, URDF)
Before this commit: robot str1ker, 7 links, 6 joints
Links:
- added link upperarm_actuator_body_link, mass 0.952544; collision mesh filename=package://str1ker/description/models/UpperArmActuatorBodyBo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; visual mesh filename=package://str1ker/description/models/UpperArmActuatorBody.s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
- added link upperarm_actuator_shaft_link, mass 0.070; collision mesh filename=package://str1ker/description/models/UpperArmActuatorShaftB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; visual mesh filename=package://str1ker/description/models/UpperArmActuatorShaft.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
Joints:
- added joint upperarm_actuator: type prismatic, parent upperarm_actuator_body_link, child upperarm_actuator_shaft_link, origin xyz=0.153 -0.002 0 rpy=0 0 0, axis 1 0 0, limit lower=-0.054 upper=-0.0005 effort=100 velocity=0.0508
- added joint upperarm_actuator_mount: type revolute, parent shoulder_link, child upperarm_actuator_body_link, origin xyz=0.101045 -0.0504975 0 rpy=0 0 0, axis 0 0 1, limit lower=1.93 upper=2.293 effort=100 velocity=1.0, mimic joint=upperarm_actuator multiplier=0.9 offset=1.560796327
- joint fixed: origin xyz=0 0 0.06 rpy=0 0 0 -> xyz=0 0 0.1 rpy=0 0 0

Commit message: Update inertial properties

File: description/robot.urdf (robot description, URDF)
Before this commit: robot str1ker, 9 links, 8 joints
Links:
- added link forearm_actuator_body_link, mass 0.76281631; collision mesh filename=package://str1ker/description/models/ForearmActuatorBodyBou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; visual mesh filename=package://str1ker/description/models/ForearmActuatorBody.stl
- link base_link: mass 0.528 -> 0.71525618
- link drumstick_link: mass 0.091 -> 0.07166651
- link forearm_link: mass 0.703 -> 0.63998399
- link shoulder_link: mass 0.36378108 -> 0.38358403
- link upperarm_actuator_body_link: mass 0.952544 -> 0.70647685
- link upperarm_actuator_shaft_link: mass 0.070 -> 0.04967122
- link upperarm_link: mass 1.139 -> 1.13853115

Commit message: Fix base offset

File: description/robot.urdf (robot description, URDF)
Before this commit: robot str1ker, 10 links, 8 joints
Links:
- removed link forearm_actuator_body_link
Joints:
- joint base: origin xyz=0 0 0.069 rpy=1.5708 0 0 -> xyz=0 0 0 rpy=1.5708 0 0

Commit message: Clean up URDF after fixing inertia

File: description/robot.urdf (robot description, URDF)
Before this commit: robot str1ker, 9 links, 8 joints
Links:
- added link forearm_actuator_body_link, mass 0.76281631; collision mesh filename=package://str1ker/description/models/ForearmActuatorBodyBou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; visual mesh filename=package://str1ker/description/models/ForearmActuatorBody.stl
- added link forearm_actuator_connector_link, mass 0.01257956; collision mesh filename=package://str1ker/description/models/ForearmActuatorConnect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; visual mesh filename=package://str1ker/description/models/ForearmActuatorConnect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
- added link forearm_actuator_shaft_link, mass 0.08789688; collision mesh filename=package://str1ker/description/models/ForearmActuatorShaftBo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; visual mesh filename=package://str1ker/description/models/ForearmActuatorShaft.s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
Joints:
- added joint forearm_actuator: type prismatic, parent forearm_actuator_body_link, child forearm_actuator_shaft_link, origin xyz=0.210 0 0 rpy=0 0 0, axis 1 0 0, limit lower=-0.0508 upper=0 effort=100 velocity=0.0109982
- added joint forearm_actuator_connector: type revolute, parent forearm_link, child forearm_actuator_connector_link, origin xyz=0.0605718 0.004 0 rpy=0 0 0, axis 0 0 1, limit lower=1.5137 upper=1.5444 effort=100 velocity=1.0, mimic joint=forearm_actuator multiplier=0.604330709 offset=1.5444
- added joint forearm_actuator_mount: type revolute, parent upperarm_link, child forearm_actuator_body_link, origin xyz=0.130 -0.034 0 rpy=0 0 0, axis 0 0 1, limit lower=-0.06 upper=0 effort=100 velocity=1.0, mimic joint=forearm_actuator multiplier=-2.5 offset=-0.146602

Commit message: Fix export error and unpause

File: description/robot.urdf (robot description, URDF)
Before this commit: robot str1ker, 12 links, 11 joints
Joints:
- joint base: origin xyz=0 0 0 rpy=1.5708 0 0 -> xyz=0 0 0.069 rpy=1.5708 0 0

Commit message: Update base link mass

File: description/robot.urdf (robot description, URDF)
Before this commit: robot str1ker, 12 links, 11 joints
Links:
- link base_link: mass 0.71525618 -> 0.70818404

Commit message: Raise robot higher

File: description/robot.urdf (robot description, URDF)
Before this commit: robot str1ker, 12 links, 11 joints
Joints:
- joint fixed: origin xyz=0 0 0.1 rpy=0 0 0 -> xyz=0 0 0.15 rpy=0 0 0

Commit message: Raise higher to avoid contact with ground

File: description/robot.urdf (robot description, URDF)
Before this commit: robot str1ker, 12 links, 11 joints
Joints:
- joint fixed: origin xyz=0 0 0.15 rpy=0 0 0 -> xyz=0 0 1 rpy=0 0 0

Commit message: Upper arm actuator working with velocity

File: description/robot.urdf (robot description, URDF)
Before this commit: robot str1ker, 12 links, 11 joints
Links:
- removed link forearm_actuator_body_link
- removed link forearm_actuator_connector_link
- removed link forearm_actuator_shaft_link
Joints:
- removed joint forearm_actuator
- removed joint forearm_actuator_connector
- removed joint forearm_actuator_mount
- joint fixed: origin xyz=0 0 1 rpy=0 0 0 -> xyz=0 0 0 rpy=0 0 0
- joint shoulder: mimic joint=upperarm_actuator multiplier=7.640691589 offset=0.817273346 -> (none)

Commit message: Add and test forearm actuator

File: description/robot.urdf (robot description, URDF)
Before this commit: robot str1ker, 9 links, 8 joints
Links:
- added link forearm_actuator_body_link, mass 0.76281631; collision mesh filename=package://str1ker/description/models/ForearmActuatorBodyBou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; visual mesh filename=package://str1ker/description/models/ForearmActuatorBody.stl
- added link forearm_actuator_shaft_link, mass 0.08789688; collision mesh filename=package://str1ker/description/models/ForearmActuatorShaftBo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; visual mesh filename=package://str1ker/description/models/ForearmActuatorShaft.s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
Joints:
- added joint forearm_actuator: type prismatic, parent forearm_actuator_body_link, child forearm_actuator_shaft_link, origin xyz=0.210 0 0 rpy=0 0 0, axis 1 0 0, limit lower=-0.0508 upper=0 effort=100 velocity=0.0109982
- added joint forearm_actuator_mount: type revolute, parent upperarm_link, child forearm_actuator_body_link, origin xyz=0.130 -0.034 0 rpy=0 0 0, axis 0 0 1, limit lower=-0.06 upper=0 effort=100 velocity=1.0, mimic joint=forearm_actuator multiplier=-2.5 offset=-0.146602

Commit message: Re-enable forearm actuator link

File: description/robot.urdf (robot description, URDF)
Before this commit: robot str1ker, 11 links, 10 joints
Links:
- added link forearm_actuator_connector_link, mass 0.01257956; collision mesh filename=package://str1ker/description/models/ForearmActuatorConnect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; visual mesh filename=package://str1ker/description/models/ForearmActuatorConnect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
Joints:
- added joint forearm_actuator_connector: type revolute, parent forearm_link, child forearm_actuator_connector_link, origin xyz=0.0605718 0.004 0 rpy=0 0 0, axis 0 0 1, limit lower=1.5137 upper=1.5444 effort=100 velocity=1.0, mimic joint=forearm_actuator multiplier=0.604330709 offset=1.5444

Commit message: Add mimic plugins experimental

File: description/robot.urdf (robot description, URDF)
Before this commit: robot str1ker, 12 links, 11 joints
Joints:
- joint shoulder: mimic (none) -> joint=upperarm_actuator multiplier=7.640691589 offset=0.817273346

Commit message: Upper arm actuator mount mimic working

File: description/robot.urdf (robot description, URDF)
Before this commit: robot str1ker, 12 links, 11 joints
Joints:
- joint upperarm_actuator_mount: limit lower=1.93 upper=2.293 effort=100 velocity=1.0 -> lower=-6 upper=6 effort=100 velocity=1.0

Commit message: Add elbow and forearm mount mimics

File: description/robot.urdf (robot description, URDF)
Before this commit: robot str1ker, 12 links, 11 joints
Joints:
- joint forearm_actuator_mount: limit lower=-0.06 upper=0 effort=100 velocity=1.0 -> lower=-6 upper=6 effort=100 velocity=1.0

Commit message: Restore solenoid geometry

File: description/robot.urdf (robot description, URDF)
Before this commit: robot str1ker, 12 links, 11 joints
Links:
- added link solenoid_mount_link, mass 0.1; collision mesh filename=package://str1ker/description/models/ArmSolenoidBoundingBox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; visual mesh filename=package://str1ker/description/models/ArmSolenoid.stl
- added link solenoid_shaft_link, mass 0.1; collision mesh filename=package://str1ker/description/models/ArmSolenoidShaftBoundi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; visual mesh filename=package://str1ker/description/models/ArmSolenoidShaft.stl
Joints:
- added joint solenoid: type prismatic, parent solenoid_mount_link, child solenoid_shaft_link, origin xyz=0 0 0 rpy=0 0 0, axis 0 0 1, limit lower=-0.0019 upper=0.001 effort=100 velocity=1.0
- added joint solenoid_mount: type revolute, parent forearm_link, child solenoid_mount_link, origin xyz=0.355 -0.031 0.013 rpy=0 0 0, axis 0 0 1, limit lower=-0.09 upper=-0.09 effort=100 velocity=1.0

Commit message: Initial solenoid state publisher implementation

File: description/robot.urdf (robot description, URDF)
Before this commit: robot str1ker, 14 links, 13 joints
Joints:
- joint solenoid_mount: type revolute -> fixed

Commit message: Debug solenoid publisher

File: description/robot.urdf (robot description, URDF)
Before this commit: robot str1ker, 14 links, 13 joints
Joints:
- joint solenoid: axis 0 0 1 -> 1 0 0

Commit message: Convert wrist to mimic

File: description/robot.urdf (robot description, URDF)
Before this commit: robot str1ker, 14 links, 13 joints
Joints:
- joint wrist: limit lower=0.959931 upper=0.959931 effort=100 velocity=1.0 -> lower=0.959931 upper=1.0 effort=100 velocity=1.0; mimic (none) -> joint=solenoid multiplier=13.8167 offset=0.9862

Commit message: Adjust config

File: description/robot.urdf (robot description, URDF)
Before this commit: robot str1ker, 14 links, 13 joints
Joints:
- joint base: limit lower=-1.4929 upper=1.4929 effort=100 velocity=1.0 -> lower=-1.5708 upper=1.5708 effort=100 velocity=1.0

Commit message: Update simulation properties

File: description/robot.urdf (robot description, URDF)
Before this commit: robot str1ker, 14 links, 13 joints
Joints:
- joint base: limit lower=-1.5708 upper=1.5708 effort=100 velocity=1.0 -> lower=-1.5708 upper=1.5708 effort=100 velocity=3.14160

Commit message: Update URDF after updating models

File: description/robot.urdf (robot description, URDF)
Before this commit: robot str1ker, 14 links, 13 joints
Joints:
- joint base: origin xyz=0 0 0.069 rpy=1.5708 0 0 -> xyz=0 0 0 rpy=1.5708 0 0
- joint fixed: origin xyz=0 0 0 rpy=0 0 0 -> xyz=0 0 0.5 rpy=0 0 0

Commit message: Fix shoulder offset in URDF

File: description/robot.urdf (robot description, URDF)
Before this commit: robot str1ker, 14 links, 13 joints
Joints:
- joint shoulder: origin xyz=-0.013 0.11518 0.0 rpy=0 0 0 -> xyz=-0.013 0.115 0.0 rpy=0 0 0

Commit message: Fix shoulder offset after re-design

File: description/robot.urdf (robot description, URDF)
Before this commit: robot str1ker, 14 links, 13 joints
Joints:
- joint shoulder: origin xyz=-0.013 0.115 0.0 rpy=0 0 0 -> xyz=-0.013 0.109 0.0 rpy=0 0 0
