File: boards/LegRobotBoardTeensy/LegRobotBoardTeensy.kicad_sch (KiCad schematic)
At the start: 50 parts, among them J1 B5B-XH-A, J10 B4B-XH-A, J11 B3B-XH-A, J2 B4B-XH-A, J3 B3B-XH-A, J4 B3B-XH-A, J5 B4B-XH-A, J6 B2B-XH-A, J7 B2B-XH-A, J8 B4B-XH-A, J9 B4B-XH-A, Q1 SMMBT3904LT1G, U1 Teensy4.0, U2 TLC555CDR, U3 SN74HC08DR, U4 SN74HC08DR

Commit message: Initial schematic
Parts:
- removed D1, D2, D3, D4, D6, D7, D9: BLUE LED, 150080BS75000:150080BS75000_Modified, symbol 150080BS75000:150080BS75000
- removed D10, D11, D5, D8: PINK LED, XL-2012UPC:LED_XL-2012SURC_XLG, symbol XL-2012UPC:XL-2012SURC
- removed J1: B5B-XH-A, Connector_JST:JST_XH_B5B-XH-A_1x05_P2.50mm_Vertical, symbol Connector_Generic:Conn_01x05
- removed J10, J2, J5, J8, J9: B4B-XH-A, Connector_JST:JST_XH_B4B-XH-A_1x04_P2.50mm_Vertical, symbol Connector_Generic:Conn_01x04
- removed J6, J7: B2B-XH-A, Connector_JST:JST_XH_B2B-XH-A_1x02_P2.50mm_Vertical, symbol Connector_Generic:Conn_01x02
- removed Q1: SMMBT3904LT1G, SMMBT3904LT1G:SMMBT3904LT1G, symbol SMMBT3904LT1G:SMMBT3904LT1G
- removed R1, R11, R2, R3, R4, R6, R7: 150R, RCG06031K00FKEA:RCG06031K00FKEA, symbol RCG06031K00FKEA:RCG06031K00FKEA
- removed R10, R12, R13, R5: 470R, RC0603FR-07470RL:RC0603FR-07470RL, symbol RCG06031K00FKEA:RCG06031K00FKEA
- removed R14, R17, R9: 100K, CRCW0603100KFKEA:CRCW0603100KFKEA, symbol CRCW0603100KFKEA:CRCW0603100KFKEA
- removed R15, R8: 10K, CRCW060310K0FKEA:CRCW060310K0FKEA, symbol CRCW060310K0FKEA:CRCW060310K0FKEA
- removed R16: 360K, RC0603FR-07360KL:RC0603FR-07360KL, symbol RC0603FR-07360KL:RC0603FR-07360KL
- added D1, D2, D3, D4, D5, D6, D7, D8: REDLED, NCD0603R1:NCD0603R1, symbol Device:LED
- added D10, D11, D12, D13, D14, D15, D16, D17, D18, D19, D20, D21, D22, D23, D24, D9: BLUELED, 150080BS75000:150080BS75000_Modified, symbol Device:LED
- added J1, J14, J15, J16: IDC, symbol Connector_Generic:Conn_02x04_Odd_Even
- added J10, J12, J13, J4, J5, J6, J7, J8, J9: B3B-XH-A, Connector_JST:JST_XH_B3B-XH-A_1x03_P2.50mm_Vertical, symbol Connector_Generic:Conn_01x03
- added Q1, Q10, Q11, Q12, Q13, Q14, Q15, Q16, Q17, Q18, Q19, Q2, Q20, Q21, Q22, Q23, Q24, Q3, Q4, Q5, Q6, Q7, Q8, Q9: MMBT3904LT1G, SMMBT3904LT1G:MMBT3904LT1G, symbol MMBT3904LT1G:MMBT3904LT1G
- added R1: 360K, RC0603FR-07360KL:RC0603FR-07360KL, symbol Device:R_US
- added R10, R3, R4, R5, R6, R7, R8, R9: 1K, RCG06031K00FKEA:RCG06031K00FKEA, symbol Device:R_US
- added R11, R12, R13, R14, R15, R16, R17, R18, R19, R20, R21, R22, R23, R24, R25, R26: 150R, RC0603FR-07150RL:RESC1607X60N, symbol Device:R_US
- added R2, R27: 10K, CRCW060310K0FKEA:CRCW060310K0FKEA, symbol Device:R_US
- added U5: PCA9685PW_118, PCA9685PW,118:PCA9685PW,118, symbol PCA9685PW,118:PCA9685PW_118
- added U6, U7: SN74HC08DR, SN74HC08DR:SN74HC08DR, symbol SN74HC08DR:SN74HC08DR
- renumbered J3 to J2, J4 to J3
Connections:
- net +3.3V: now also J1.1 (Pin_1), J14.1 (Pin_1), J15.1 (Pin_1), J16.1 (Pin_1), J4.1 (Pin_1), J5.1 (Pin_1), R10.2, R11.2, R12.2, R13.2, R14.2, R15.2, R16.2, R17.2, R18.2, R19.2, R2.1, R20.2, R21.2, R22.2, R23.2, R24.2, R25.2, R26.2, R3.2, R4.2, R5.2, R6.2, R7.2, R8.2, R9.2, U5.28 (VDD), U6.14 (VCC), U7.14 (VCC); no longer J11.2 (Pin_2)
- net BLINK: now also U4.12 (4A), U4.9 (3A), U6.1 (1A), U6.12 (4A), U6.4 (2A), U6.9 (3A), U7.1 (1A), U7.12 (4A), U7.4 (2A), U7.9 (3A)
- net GND: now also U1.17 (GND), U1.47 (GND), J1.2 (Pin_2), J1.4 (Pin_4), J1.6 (Pin_6), J1.8 (Pin_8), J14.2 (Pin_2), J14.4 (Pin_4), J14.6 (Pin_6), J14.8 (Pin_8), J15.2 (Pin_2), J15.4 (Pin_4), J15.6 (Pin_6), J15.8 (Pin_8), J16.2 (Pin_2), J16.4 (Pin_4), J16.6 (Pin_6), J16.8 (Pin_8), J4.3 (Pin_3), J5.3 (Pin_3), Q1.2 (E), Q10.2 (E), Q11.2 (E), Q12.2 (E), Q13.2 (E), Q14.2 (E), Q15.2 (E), Q16.2 (E), Q17.2 (E), Q18.2 (E), Q19.2 (E), Q2.2 (E), Q20.2 (E), Q21.2 (E), Q22.2 (E), Q23.2 (E), Q24.2 (E), Q3.2 (E), Q4.2 (E), Q5.2 (E), Q6.2 (E), Q7.2 (E), Q8.2 (E), Q9.2 (E), R27.2, U5.1 (A0), U5.14 (VSS), U5.2 (A1), U5.24 (A5), U5.25 (EXTCLK), U5.3 (A2), U5.4 (A3), U5.5 (A4), U6.7 (GND), U7.7 (GND); no longer J11.3 (Pin_3)
- net LPWM1: now also J6.3 (Pin_3), U5.7 (LED1); no longer U1.5 (3_LRCLK2)
- net LPWM2: now also J7.3 (Pin_3), U5.9 (LED3); no longer U1.10 (8_TX2_IN1)
- net LPWM3: now also J8.3 (Pin_3), U5.11 (LED5); no longer U1.30 (23_A9_CRX1_MCLK1)
- net NODE_A: now also R1.1
- net NODE_B: now also R1.2, R2.2
- net RPWM1: now also J6.2 (Pin_2), U5.6 (LED0); no longer U1.3 (1_TX1_CTX2_MISO1)
- net RPWM2: now also J7.2 (Pin_2), U5.8 (LED2); no longer U1.9 (7_RX2_OUT1A)
- net RPWM3: now also J8.2 (Pin_2), U5.10 (LED4); no longer U1.29 (22_A8_CTX1)
- net SCL: now also U5.26 (SCL)
- net SDA: now also U5.27 (SDA)
- net PWMEN4: now reaches U1.13 (11_MOSI_CTX1)
- net PWMEN4: now also J9.1 (Pin_1), Q4.1 (B)
- net LPWM4: now reaches U4.10 (3B)
- net LPWM4: now also J9.3 (Pin_3), U5.13 (LED7)
- net RPWM4BLINK: now reaches U4.11 (4Y)
- net RPWM4BLINK: now also Q15.1 (B)
- net RPWM4: now reaches U4.13 (4B)
- net RPWM4: now also J9.2 (Pin_2), U5.12 (LED6)
- net LPWM4BLINK: now reaches U4.8 (3Y)
- net LPWM4BLINK: now also Q16.1 (B)
- net A renamed ENCODER2_A
- net ENCODER2_A: now also J14.3 (Pin_3)
- net B renamed ENCODER3_B
- net ENCODER3_B: now also J15.5 (Pin_5)
- net CS renamed PWMEN3
- net PWMEN3: now also J8.1 (Pin_1), Q3.1 (B)
- net LPWM1A renamed LPWM1BLINK
- net LPWM1BLINK: now also Q10.1 (B)
- net LPWM2A renamed LPWM2BLINK
- net LPWM2BLINK: now also Q12.1 (B)
- net LPWM3A renamed LPWM3BLINK
- net LPWM3BLINK: now also Q14.1 (B)
- net MISO renamed PWMEN5
- net PWMEN5: now also J10.1 (Pin_1), Q5.1 (B)
- net PWM1EN renamed ENCODER1_A
- net ENCODER1_A: now also J1.3 (Pin_3)
- net PWM1VT renamed A2
- net A2: now also J4.2 (Pin_2)
- net PWM2EN renamed PWMEN1
- net PWMEN1: now also J6.1 (Pin_1), Q1.1 (B)
- net PWM2VT renamed ENCODER3_A
- net ENCODER3_A: now also J15.3 (Pin_3)
- net PWM3EN renamed PWMEN8
- net PWMEN8: now also J13.1 (Pin_1), Q8.1 (B)
- net PWM3VT renamed PWMEN7
- net PWMEN7: now also J12.1 (Pin_1), Q7.1 (B)
- net RPWM1A renamed RPWM1BLINK
- net RPWM1BLINK: now also Q9.1 (B)
- net RPWM2A renamed RPWM2BLINK
- net RPWM2BLINK: now also Q11.1 (B)
- net RPWM3A renamed RPWM3BLINK
- net RPWM3BLINK: now also Q13.1 (B)
- net SCK renamed PWMEN6
- net PWMEN6: now also J11.1 (Pin_1), Q6.1 (B)
- net SIG renamed A3
- net A3: now also J5.2 (Pin_2); no longer J11.1 (Pin_1)
- net SPIS renamed PWMEN2
- net PWMEN2: now also J7.1 (Pin_1), Q2.1 (B)
- new net: D17.2 (A), R19.1
- new net: D1.2 (A), R3.1
- new net: D8.2 (A), R10.1
- new net: D23.1 (K), Q23.3 (C)
- new net: R27.1, U5.23 (*OE)
- new net: D2.1 (K), Q2.3 (C)
- new net: D19.2 (A), R21.1
- new net: D15.1 (K), Q15.3 (C)
- new net: D15.2 (A), R17.1
- new net: D9.2 (A), R11.1
- new net: D5.1 (K), Q5.3 (C)
- new net: D7.2 (A), R9.1
- new net: D17.1 (K), Q17.3 (C)
- new net: D16.1 (K), Q16.3 (C)
- new net: D5.2 (A), R7.1
- new net: D4.2 (A), R6.1
- new net: D19.1 (K), Q19.3 (C)
- new net: D11.1 (K), Q11.3 (C)
- new net: D12.2 (A), R14.1
- new net: D21.1 (K), Q21.3 (C)
- new net: D22.2 (A), R24.1
- new net: D3.1 (K), Q3.3 (C)
- new net: D8.1 (K), Q8.3 (C)
- new net: D16.2 (A), R18.1
- new net: D13.1 (K), Q13.3 (C)
- new net: D3.2 (A), R5.1
- new net: D10.1 (K), Q10.3 (C)
- new net: D2.2 (A), R4.1
- new net: D6.1 (K), Q6.3 (C)
- new net: D6.2 (A), R8.1
- new net: D20.1 (K), Q20.3 (C)
- new net: D20.2 (A), R22.1
- new net: D11.2 (A), R13.1
- new net: D7.1 (K), Q7.3 (C)
- new net: D1.1 (K), Q1.3 (C)
- new net: D14.1 (K), Q14.3 (C)
- new net: D18.1 (K), Q18.3 (C)
- new net: D24.1 (K), Q24.3 (C)
- new net: D24.2 (A), R26.1
- new net: D12.1 (K), Q12.3 (C)
- new net: D14.2 (A), R16.1
- new net: D13.2 (A), R15.1
- new net: D9.1 (K), Q9.3 (C)
- new net: D21.2 (A), R23.1
- new net: D22.1 (K), Q22.3 (C)
- new net: D10.2 (A), R12.1
- new net: D23.2 (A), R25.1
- new net: D4.1 (K), Q4.3 (C)
- new net: D18.2 (A), R20.1
- new net ENCODER1_B: J1.5 (Pin_5), U1.3 (1_TX1_CTX2_MISO1)
- new net ENCODER1_I: J1.7 (Pin_7)
- new net ENCODER2_B: J14.5 (Pin_5), U1.5 (3_LRCLK2)
- new net ENCODER2_I: J14.7 (Pin_7)
- new net ENCODER3_I: J15.7 (Pin_7)
- new net ENCODER4_A: J16.3 (Pin_3), U1.9 (7_RX2_OUT1A)
- new net ENCODER4_B: J16.5 (Pin_5), U1.10 (8_TX2_IN1)
- new net ENCODER4_I: J16.7 (Pin_7)
- new net LPWM5: J10.3 (Pin_3), U5.16 (LED9), U6.5 (2B)
- new net LPWM5BLINK: Q18.1 (B), U6.6 (2Y)
- new net LPWM6: J11.3 (Pin_3), U5.18 (LED11), U6.10 (3B)
- new net LPWM6BLINK: Q20.1 (B), U6.8 (3Y)
- new net LPWM7: J12.3 (Pin_3), U5.20 (LED13), U7.5 (2B)
- new net LPWM7BLINK: Q22.1 (B), U7.6 (2Y)
- new net LPWM8: J13.3 (Pin_3), U5.22 (LED15), U7.10 (3B)
- new net LPWM8BLINK: Q24.1 (B), U7.8 (3Y)
- new net RPWM5: J10.2 (Pin_2), U5.15 (LED8), U6.2 (1B)
- new net RPWM5BLINK: Q17.1 (B), U6.3 (1Y)
- new net RPWM6: J11.2 (Pin_2), U5.17 (LED10), U6.13 (4B)
- new net RPWM6BLINK: Q19.1 (B), U6.11 (4Y)
- new net RPWM7: J12.2 (Pin_2), U5.19 (LED12), U7.2 (1B)
- new net RPWM7BLINK: Q21.1 (B), U7.3 (1Y)
- new net RPWM8: J13.2 (Pin_2), U5.21 (LED14), U7.13 (4B)
- new net RPWM8BLINK: Q23.1 (B), U7.11 (4Y)
- no-connect marks 39 -> 32
Other:
- note added: "555 Timer"
- note added: "ADC"
- note added: "Controller"
- note added: "Gates"
- note added: "LPWM / RPWM"
- note added: "LPWM 1"
- note added: "LPWM 2"
- note added: "LPWM 3"
- note added: "LPWM 4"
- note added: "LPWM 5"
- note added: "LPWM 6"
- note added: "LPWM 7"
- note added: "LPWM 8"
- note added: "Mount Holes"
- note added: "PWM"
- note added: "PWM 1"
- note added: "PWM 2"
- note added: "PWM 3"
- note added: "PWM 4"
- note added: "PWM 5"
- note added: "PWM 6"
- note added: "PWM 7"
- note added: "PWM 8"
- note added: "PWM Driver"
- note added: "PWM ENABLED"
- note added: "QUADRATURE"
- note added: "RPWM 1"
- note added: "RPWM 2"
- note added: "RPWM 3"
- note added: "RPWM 4"
- note added: "RPWM 5"
- note added: "RPWM 6"
- note added: "RPWM 7"
- note added: "RPWM 8"
- note removed: "01 Binary : Tech Art"
- note removed: "TEENSY MOTOR CONTROL BOARD"
- moved on the sheet: C1, C2, J2, J3, MH1, MH2, MH3, MH4, U1, U2, U3, U4
