File: boards/LegRobotBoardTeensy/LegRobotBoardTeensy.kicad_sch (KiCad schematic)
At the start: 108 parts, among them J1 IDC, J10 B3B-XH-A, J11 B3B-XH-A, J12 B3B-XH-A, J13 B3B-XH-A, J14 IDC, J15 IDC, J16 IDC, J2 B3B-XH-A, J3 B3B-XH-A, J4 B3B-XH-A, J5 B3B-XH-A, J6 B3B-XH-A, J7 B3B-XH-A, J8 B3B-XH-A, J9 B3B-XH-A, Q1 MMBT3904LT1G, Q10 MMBT3904LT1G, Q11 MMBT3904LT1G, Q12 MMBT3904LT1G, Q13 MMBT3904LT1G, Q14 MMBT3904LT1G, Q15 MMBT3904LT1G, Q16 MMBT3904LT1G, Q17 MMBT3904LT1G, Q18 MMBT3904LT1G, Q19 MMBT3904LT1G, Q2 MMBT3904LT1G, Q20 MMBT3904LT1G, Q21 MMBT3904LT1G, Q22 MMBT3904LT1G, Q23 MMBT3904LT1G, Q24 MMBT3904LT1G, Q3 MMBT3904LT1G, Q4 MMBT3904LT1G, Q5 MMBT3904LT1G, Q6 MMBT3904LT1G, Q7 MMBT3904LT1G, Q8 MMBT3904LT1G, Q9 MMBT3904LT1G, U1 Teensy4.0, U2 TLC555CDR, U3 SN74HC08DR, U4 SN74HC08DR, U5 PCA9685PW_118, U6 SN74HC08DR, U7 SN74HC08DR, U8 BNO055

Commit message: Update main and leg board
Parts:
- removed J10, J11, J12, J13, J6, J7, J8, J9: B3B-XH-A, Connector_JST:JST_XH_B3B-XH-A_1x03_P2.50mm_Vertical, symbol Connector_Generic:Conn_01x03
- added C5, C6, C7, C8: 47nF, CL10B473KB8NNNC:CAPC1608X90N, symbol CC0603JRX7R7BB105:CC0603JRX7R7BB105
- added J10, J11, J12, J13, J6, J7, J8, J9: IDC, Connector_IDC:IDC-Header_2x04_P2.54mm_Vertical, symbol Connector_Generic:Conn_02x04_Odd_Even
- added R29, R30, R31, R32: 2.2K, RC0603FR-072K2L:RC0603FR-072K2L, symbol Device:R_US
Connections:
- net +3.3V: now also J10.2 (Pin_2), J11.2 (Pin_2), J12.2 (Pin_2), J13.2 (Pin_2), J6.2 (Pin_2), J7.2 (Pin_2), J8.2 (Pin_2), J9.2 (Pin_2)
- net A0: now also R29.2; no longer J2.2 (Pin_2)
- net A1: now also R30.2; no longer J3.2 (Pin_2)
- net A2: now also R31.2; no longer J4.2 (Pin_2)
- net A3: now also R32.2; no longer J5.2 (Pin_2)
- net GND: now also C5.1, C6.1, C7.1, C8.1, J10.1 (Pin_1), J11.1 (Pin_1), J12.1 (Pin_1), J13.1 (Pin_1), J6.1 (Pin_1), J7.1 (Pin_1), J8.1 (Pin_1), J9.1 (Pin_1)
- net LPWM1: now also J6.7 (Pin_7)
- net LPWM2: now also J7.7 (Pin_7)
- net LPWM3: now also J8.7 (Pin_7)
- net LPWM4: now also J9.7 (Pin_7)
- net LPWM5: now also J10.7 (Pin_7)
- net LPWM6: now also J11.7 (Pin_7)
- net LPWM7: now also J12.7 (Pin_7)
- net LPWM8: now also J13.7 (Pin_7)
- net PWMEN1: now also J6.5 (Pin_5), J6.6 (Pin_6)
- net PWMEN2: now also J7.5 (Pin_5), J7.6 (Pin_6)
- net PWMEN3: now also J8.5 (Pin_5), J8.6 (Pin_6)
- net PWMEN4: now also J9.5 (Pin_5), J9.6 (Pin_6)
- net PWMEN5: now also J10.5 (Pin_5), J10.6 (Pin_6)
- net PWMEN6: now also J11.5 (Pin_5), J11.6 (Pin_6)
- net PWMEN7: now also J12.5 (Pin_5), J12.6 (Pin_6)
- net PWMEN8: now also J13.5 (Pin_5), J13.6 (Pin_6)
- net RPWM1: now also J6.8 (Pin_8)
- net RPWM2: now also J7.8 (Pin_8)
- net RPWM3: now also J8.8 (Pin_8)
- net RPWM4: now also J9.8 (Pin_8)
- net RPWM5: now also J10.8 (Pin_8)
- net RPWM6: now also J11.8 (Pin_8)
- net RPWM7: now also J12.8 (Pin_8)
- net RPWM8: now also J13.8 (Pin_8)
- new net: C6.2, J3.2 (Pin_2), R30.1
- new net: C7.2, J4.2 (Pin_2), R31.1
- new net: C5.2, J2.2 (Pin_2), R29.1
- new net: C8.2, J5.2 (Pin_2), R32.1
- new net L_IS1: J6.3 (Pin_3)
- new net L_IS2: J7.3 (Pin_3)
- new net L_IS3: J8.3 (Pin_3)
- new net L_IS4: J9.3 (Pin_3)
- new net L_IS5: J10.3 (Pin_3)
- new net L_IS6: J11.3 (Pin_3)
- new net L_IS7: J12.3 (Pin_3)
- new net L_IS8: J13.3 (Pin_3)
- new net R_IS1: J6.4 (Pin_4)
- new net R_IS2: J7.4 (Pin_4)
- new net R_IS3: J8.4 (Pin_4)
- new net R_IS4: J9.4 (Pin_4)
- new net R_IS5: J10.4 (Pin_4)
- new net R_IS6: J11.4 (Pin_4)
- new net R_IS7: J12.4 (Pin_4)
- new net R_IS8: J13.4 (Pin_4)
Other:
- note added: "CONTROLLER"
- note added: "GATES"
- note added: "INDICATORS"
- note added: "PWM DRIVER"
- note removed: "Controller"
- note removed: "Gates"
- note removed: "PWM Driver"
- moved on the sheet: C1, C2, C3, C4, D1, D10, D11, D12, D13, D14, D15, D16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

Commit message: Minor normalization
Parts:
- C2: value 0.01uF -> 10nF
Changed lines of the file:
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@@
 			)
 		)
-		(property "Value" "0.01uF"
+		(property "Value" "10nF"
 			(at 511.302 118.618 0)
 			(effects

Commit message: Update leg encoder board and documentation
Parts:
- added R33, R36, R37, R39, R41, R43, R45, R47, R49, R51, R53, R55, R57, R59, R61, R63, R65, R67, R69, R71, R73, R75, R77, R81: 10K, CRCW060310K0FKEA:CRCW060310K0FKEA, symbol Device:R_US
- added R34, R35, R38, R40, R42, R44, R46, R48, R50, R52, R54, R56, R58, R60, R62, R64, R66, R68, R70, R72, R74, R76, R78, R80: 100K, CRCW0603100KFKEA:CRCW0603100KFKEA, symbol Device:R_US
Connections:
- net GND: now also R34.2, R35.2, R38.2, R40.2, R42.2, R44.2, R46.2, R48.2, R50.2, R52.2, R54.2, R56.2, R58.2, R60.2, R62.2, R64.2, R66.2, R68.2, R70.2, R72.2, R74.2, R76.2, R78.2, R80.2
- net LPWM1BLINK: now also R49.1, R52.1; no longer Q10.1 (B)
- net LPWM2BLINK: now also R75.1, R76.1; no longer Q12.1 (B)
- net LPWM3BLINK: now also R51.1, R54.1; no longer Q14.1 (B)
- net LPWM4BLINK: now also R73.1, R74.1; no longer Q16.1 (B)
- net LPWM5BLINK: now also R53.1, R56.1; no longer Q18.1 (B)
- net LPWM6BLINK: now also R71.1, R72.1; no longer Q20.1 (B)
- net LPWM7BLINK: now also R55.1, R58.1; no longer Q22.1 (B)
- net LPWM8BLINK: now also R57.1, R60.1; no longer Q24.1 (B)
- net PWMEN1: now also R34.1, R81.1; no longer Q1.1 (B)
- net PWMEN2: now also R45.1, R48.1; no longer Q2.1 (B)
- net PWMEN3: now also R59.1, R62.1; no longer Q3.1 (B)
- net PWMEN4: now also R69.1, R80.1; no longer Q4.1 (B)
- net PWMEN5: now also R33.1, R35.1; no longer Q5.1 (B)
- net PWMEN6: now also R47.1, R50.1; no longer Q6.1 (B)
- net PWMEN7: now also R61.1, R64.1; no longer Q7.1 (B)
- net PWMEN8: now also R77.1, R78.1; no longer Q8.1 (B)
- net RPWM1BLINK: now also R36.1, R38.1; no longer Q9.1 (B)
- net RPWM2BLINK: now also R63.1, R66.1; no longer Q11.1 (B)
- net RPWM3BLINK: now also R37.1, R40.1; no longer Q13.1 (B)
- net RPWM4BLINK: now also R65.1, R68.1; no longer Q15.1 (B)
- net RPWM5BLINK: now also R39.1, R42.1; no longer Q17.1 (B)
- net RPWM6BLINK: now also R67.1, R70.1; no longer Q19.1 (B)
- net RPWM7BLINK: now also R41.1, R44.1; no longer Q21.1 (B)
- net RPWM8BLINK: now also R43.1, R46.1; no longer Q23.1 (B)
- new net: Q17.1 (B), R39.2
- new net: Q23.1 (B), R43.2
- new net: Q2.1 (B), R45.2
- new net: Q24.1 (B), R57.2
- new net: Q16.1 (B), R73.2
- new net: Q5.1 (B), R33.2
- new net: Q14.1 (B), R51.2
- new net: Q11.1 (B), R63.2
- new net: Q4.1 (B), R69.2
- new net: Q21.1 (B), R41.2
- new net: Q3.1 (B), R59.2
- new net: Q8.1 (B), R77.2
- new net: Q18.1 (B), R53.2
- new net: Q13.1 (B), R37.2
- new net: Q22.1 (B), R55.2
- new net: Q7.1 (B), R61.2
- new net: Q10.1 (B), R49.2
- new net: Q9.1 (B), R36.2
- new net: Q6.1 (B), R47.2
- new net: Q1.1 (B), R81.2
- new net: Q12.1 (B), R75.2
- new net: Q19.1 (B), R67.2
- new net: Q15.1 (B), R65.2
- new net: Q20.1 (B), R71.2
Other:
- moved on the sheet: C1, C2, C3, C4, C5, C6, C7, C8, D1, D10, D11, D12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

Commit message: Second iteration of leg robot board
Parts:
- removed Q1, Q10, Q11, Q12, Q13, Q14, Q15, Q16, Q17, Q18, Q19, Q2, Q20, Q21, Q22, Q23, Q24, Q3, Q4, Q5, Q6, Q7, Q8, Q9: MMBT3904LT1G, SMMBT3904LT1G:MMBT3904LT1G, symbol MMBT3904LT1G:MMBT3904LT1G
- added Q1, Q10, Q11, Q12, Q13, Q14, Q15, Q16, Q17, Q18, Q19, Q2, Q20, Q21, Q22, Q23, Q24, Q3, Q4, Q5, Q6, Q7, Q8, Q9: AO3400A, AO3400A:AO3400A, symbol AO3400A:AO3400A
Connections:
- net GND: now also Q1.3, Q10.3, Q11.3, Q12.3, Q13.3, Q14.3, Q15.3, Q16.3, Q17.3, Q18.3, Q19.3, Q2.3, Q20.3, Q21.3, Q22.3, Q23.3, Q24.3, Q3.3, Q4.3, Q5.3, Q6.3, Q7.3, Q8.3, Q9.3
- net at R39.2: now also Q17.1
- net at R43.2: now also Q23.1
- net at D23.1 (K): now also Q23.2
- net at R45.2: now also Q2.1
- net at D2.1 (K): now also Q2.2
- net at D15.1 (K): now also Q15.2
- net at R57.2: now also Q24.1
- net at R73.2: now also Q16.1
- net at R33.2: now also Q5.1
- net at D5.1 (K): now also Q5.2
- net at D17.1 (K): now also Q17.2
- net at R51.2: now also Q14.1
- net at D16.1 (K): now also Q16.2
- net at D19.1 (K): now also Q19.2
- net at R63.2: now also Q11.1
- net at R69.2: now also Q4.1
- net at D11.1 (K): now also Q11.2
- net at R41.2: now also Q21.1
- net at D21.1 (K): now also Q21.2
- net at R59.2: now also Q3.1
- net at D3.1 (K): now also Q3.2
- net at R77.2: now also Q8.1
- net at R53.2: now also Q18.1
- net at D8.1 (K): now also Q8.2
- net at R37.2: now also Q13.1
- net at D13.1 (K): now also Q13.2
- net at R55.2: now also Q22.1
- net at R61.2: now also Q7.1
- net at R49.2: now also Q10.1
- net at D10.1 (K): now also Q10.2
- net at R36.2: now also Q9.1
- net at D6.1 (K): now also Q6.2
- net at R47.2: now also Q6.1
- net at D20.1 (K): now also Q20.2
- net at D7.1 (K): now also Q7.2
- net at R81.2: now also Q1.1
- net at D1.1 (K): now also Q1.2
- net at R75.2: now also Q12.1
- net at D14.1 (K): now also Q14.2
- net at D18.1 (K): now also Q18.2
- net at D24.1 (K): now also Q24.2
- net at D12.1 (K): now also Q12.2
- net at R67.2: now also Q19.1
- net at D9.1 (K): now also Q9.2
- net at D22.1 (K): now also Q22.2
- net at R65.2: now also Q15.1
- net at D4.1 (K): now also Q4.2
- net at R71.2: now also Q20.1
Other:
- note added: "MOUNT HOLES"
- note removed: "Mount Holes"

Commit message: Order legs board
Parts:
- C5, C6, C7, C8: LCSC (none) -> C1622
- R29, R30, R31, R32: LCSC (none) -> C114662
Connections:
- no-connect marks 28 -> 29
Changed lines of the file:
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@@
 	)
 	(no_connect
+		(at 326.39 57.15)
+	)
+	(no_connect
 		(at 284.48 57.15)
 	)
@@
 			)
 		)
-		(property "LCSC" ""
+		(property "LCSC" "C1622"
 			(at 176.5299 35.56 0)
 			(effects
@@
 			)
 		)
-		(property "LCSC" ""
+		(property "LCSC" "C114662"
 			(at 187.96 30.48 0)
 			(effects
@@
 			)
 		)
-		(property "LCSC" ""
+		(property "LCSC" "C114662"
 			(at 187.96 66.04 0)
 			(effects
@@
 			)
 		)
-		(property "LCSC" ""
+		(property "LCSC" "C1622"
 			(at 176.5299 88.9 0)
 			(effects
@@
 			)
 		)
-		(property "LCSC" ""
+		(property "LCSC" "C114662"
 			(at 187.96 83.82 0)
 			(effects
@@
 			)
 		)
-		(property "LCSC" ""
+		(property "LCSC" "C1622"
 			(at 176.5299 53.34 0)
 			(effects
@@
 			)
 		)
-		(property "LCSC" ""
+		(property "LCSC" "C1622"
 			(at 176.5299 71.12 0)
 			(effects
@@
 			)
 		)
-		(property "LCSC" ""
+		(property "LCSC" "C114662"
 			(at 187.96 48.26 0)
 			(effects

Commit message: Add LED number displays to legs board and re-finalize
Parts:
- added C10: 10nF, C0402C103J4RACTU:C0402C103J4RACTU, symbol C0402C103J4RACTU:C0402C103J4RACTU
- added C9: 100nF, CC0603KRX7R9BB104:CC0603KRX7R9BB104, symbol CC0603KRX7R9BB104:CC0603KRX7R9BB104
- added J17, J18, J19, J20, J21, J22, J23, J24: Conn_01x05, Connector_PinHeader_2.54mm:PinHeader_1x05_P2.54mm_Vertical, symbol Connector_Generic:Conn_01x05
- added R79, R82: 4.7K, CR0603-FX-4701ELF:CR0603-FX-4701ELF, symbol Device:R_US
- added U9: HT16K33A-28SSOP, LCDDriver:HT16K33A-28SSOP, symbol LCDDriver:HT16K33A-28SSOP
Connections:
- net +3.3V: now also C10.1, C9.1, R79.1, R82.1, U9.28 (VDD)
- net GND: now also Q1.2, Q10.2, Q11.2, Q12.2, Q13.2, Q14.2, Q15.2, Q16.2, Q17.2, Q18.2, Q19.2, Q2.2, Q20.2, Q21.2, Q22.2, Q23.2, Q24.2, Q3.2, Q4.2, Q5.2, Q6.2, Q7.2, Q8.2, Q9.2, C10.2, C9.2, U9.1 (VSS); no longer Q1.3, Q10.3, Q11.3, Q12.3, Q13.3, Q14.3, Q15.3, Q16.3, Q17.3, Q18.3, Q19.3, Q2.3, Q20.3, Q21.3, Q22.3, Q23.3, Q24.3, Q3.3, Q4.3, Q5.3, Q6.3, Q7.3, Q8.3, Q9.3
- net SCL: now also R79.2, U9.26 (SCL)
- net SDA: now also R82.2, U9.27 (SDA)
- net at D21.1 (K): now also Q21.3; no longer Q21.2
- net at D15.1 (K): now also Q15.3; no longer Q15.2
- net at D18.1 (K): now also Q18.3; no longer Q18.2
- net at D12.1 (K): now also Q12.3; no longer Q12.2
- net at D9.1 (K): now also Q9.3; no longer Q9.2
- net at D22.1 (K): now also Q22.3; no longer Q22.2
- net at D5.1 (K): now also Q5.3; no longer Q5.2
- net at D13.1 (K): now also Q13.3; no longer Q13.2
- net at D1.1 (K): now also Q1.3; no longer Q1.2
- net at D19.1 (K): now also Q19.3; no longer Q19.2
- net at D14.1 (K): now also Q14.3; no longer Q14.2
- net at D8.1 (K): now also Q8.3; no longer Q8.2
- net at D4.1 (K): now also Q4.3; no longer Q4.2
- net at D16.1 (K): now also Q16.3; no longer Q16.2
- net at D10.1 (K): now also Q10.3; no longer Q10.2
- net at D23.1 (K): now also Q23.3; no longer Q23.2
- net at D6.1 (K): now also Q6.3; no longer Q6.2
- net at D20.1 (K): now also Q20.3; no longer Q20.2
- net at D11.1 (K): now also Q11.3; no longer Q11.2
- net at D17.1 (K): now also Q17.3; no longer Q17.2
- net at D7.1 (K): now also Q7.3; no longer Q7.2
- net at D3.1 (K): now also Q3.3; no longer Q3.2
- net at D24.1 (K): now also Q24.3; no longer Q24.2
- net at D2.1 (K): now also Q2.3; no longer Q2.2
- new net COM0: J18.5 (Pin_5), U9.2 (COM0/AD)
- new net COM1: J17.5 (Pin_5), U9.3 (COM1/KS0)
- new net COM2: J19.5 (Pin_5), U9.4 (COM2/KS1)
- new net COM3: J20.5 (Pin_5), U9.5 (COM3/KS2)
- new net COM4: J21.5 (Pin_5), U9.6 (COM4)
- new net COM5: J22.5 (Pin_5), U9.7 (COM5)
- new net COM6: J23.5 (Pin_5), U9.8 (COM6)
- new net COM7: J24.5 (Pin_5), U9.9 (COM7)
- new net DIGIT_A: J17.3 (Pin_3), J20.3 (Pin_3), J22.3 (Pin_3), J24.3 (Pin_3), U9.25 (ROW0/A2)
- new net DIGIT_B: J18.4 (Pin_4), J19.4 (Pin_4), J21.4 (Pin_4), J23.4 (Pin_4), U9.24 (ROW1/A1)
- new net DIGIT_C: J18.3 (Pin_3), J19.3 (Pin_3), J21.3 (Pin_3), J23.3 (Pin_3), U9.23 (ROW2/A0)
- new net DIGIT_D: J18.1 (Pin_1), J19.1 (Pin_1), J21.1 (Pin_1), J23.1 (Pin_1), U9.22 (ROW3/K1)
- new net DIGIT_DP: J17.2 (Pin_2), J20.2 (Pin_2), J22.2 (Pin_2), J24.2 (Pin_2)
- new net DIGIT_E: J18.2 (Pin_2), J19.2 (Pin_2), J21.2 (Pin_2), J23.2 (Pin_2), U9.21 (ROW4/K2)
- new net DIGIT_F: J17.4 (Pin_4), J20.4 (Pin_4), J22.4 (Pin_4), J24.4 (Pin_4), U9.20 (ROW5/K3)
- new net DIGIT_G: J17.1 (Pin_1), J20.1 (Pin_1), J22.1 (Pin_1), J24.1 (Pin_1), U9.19 (ROW6/K4)
- no-connect marks 29 -> 38
Other:
- note added: "2-DIGIT WHEEL SPEED LED DISPLAYS"
- note added: "FRONT LEFT"
- note added: "FRONT RIGHT"
- note added: "LED DISPLAYS"
- note added: "LED MUX"
- note added: "LOGIC GATES"
- note added: "LPWM / RPWM ACTIVITY BLINKING LEDS"
- note added: "MCU"
- note added: "PWM ENABLED LEDS"
- note added: "REAR LEFT"
- note added: "REAR RIGHT"
- note removed: "CONTROLLER"
- note removed: "GATES"
- note removed: "LPWM / RPWM"
- note removed: "PWM ENABLED"
- company: (none) -> 01 Binary
- title: (none) -> Leg Robot Board
- moved on the sheet: C1, C2, C3, C4, C5, C6, C7, C8, D1, D10, D11, D12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

Commit message: Preflight leg robot board
Parts:
- R79, R82: LCSC (none) -> C17673
Changed lines of the file:
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@@
 			)
 		)
-		(property "LCSC" ""
+		(property "LCSC" "C17673"
 			(at 69.85 342.9 0)
 			(effects
@@
 			)
 		)
-		(property "LCSC" ""
+		(property "LCSC" "C17673"
 			(at 87.63 340.36 0)
 			(effects

Commit message: Re-order leg board with different LED control chip
Parts:
- removed U9: HT16K33A-28SSOP, LCDDriver:HT16K33A-28SSOP, symbol LCDDriver:HT16K33A-28SSOP
- added R83: 10K, CRCW060310K0FKEA:CRCW060310K0FKEA, symbol Device:R_US
- added R84: 20K, CRCW060310K0FKEA:CRCW060310K0FKEA, symbol Device:R_US
- added U11: IS31FL3739-GRLS4-TR, IS31FL3730-QFLS2-TR:IS31FL3730-QFLS2-TR, symbol IS31FL3730-QFLS2-TR:IS31FL3739-GRLS4-TR
- C10: value 10nF -> 1uF; footprint C0402C103J4RACTU:C0402C103J4RACTU -> CC0603JRX7R7BB105:CC0603JRX7R7BB105
Connections:
- net +3.3V: now also R83.1, U11.3 (VCC)
- net COM0: now also U11.2 (SW1)
- net COM1: now also U11.1 (SW2)
- net COM2: now also U11.24 (SW3)
- net COM3: now also U11.23 (SW4)
- net COM4: now also U11.22 (SW5)
- net COM5: now also U11.21 (SW6)
- net COM6: now also U11.20 (SW7)
- net COM7: now also U11.19 (SW8)
- net DIGIT_A: now also U11.10 (CS1)
- net DIGIT_B: now also U11.11 (CS2)
- net DIGIT_C: now also U11.12 (CS3)
- net DIGIT_D: now also U11.13 (CS4)
- net DIGIT_DP: now also U11.18 (SW9/CS8)
- net DIGIT_E: now also U11.14 (CS5)
- net DIGIT_F: now also U11.16 (CS6)
- net DIGIT_G: now also U11.17 (CS7)
- net GND: now also R84.1, U11.15 (GND), U11.4 (GND), U11.9 (AD)
- net SCL: now also U11.7 (SCL)
- net SDA: now also U11.6 (SDA)
- net RST: no longer names the net of R28.1, U8.RST
- net RST: no longer U1.37 (26_A12_MOSI1)
- new net: R83.2, U11.8 (SDB)
- new net: R84.2, U11.5 (ISET)
- no-connect marks 38 -> 30
Other:
- moved on the sheet: C10, C9, J17, J18, J19, J20, J21, J22, J23, J24, R79, R82
