File: boards/LegRobotBoardTeensy/LegRobotBoardTeensy.kicad_sch (KiCad schematic)
At the start: 173 parts, among them J1 IDC, J10 IDC, J11 IDC, J12 IDC, J13 IDC, J14 IDC, J15 IDC, J16 IDC, J17 Conn_01x10, J18 Conn_01x10, J19 Conn_01x10, J2 B3B-XH-A, J20 Conn_01x10, J3 B3B-XH-A, J4 B3B-XH-A, J5 B3B-XH-A, J6 IDC, J7 IDC, J8 IDC, J9 IDC, Q1 AO3400A, Q10 AO3400A, Q11 AO3400A, Q12 AO3400A, Q13 AO3400A, Q14 AO3400A, Q15 AO3400A, Q16 AO3400A, Q17 AO3400A, Q18 AO3400A, Q19 AO3400A, Q2 AO3400A, Q20 AO3400A, Q21 AO3400A, Q22 AO3400A, Q23 AO3400A, Q24 AO3400A, Q3 AO3400A, Q4 AO3400A, Q5 AO3400A, Q6 AO3400A, Q7 AO3400A, Q8 AO3400A, Q9 AO3400A, U1 Teensy4.1, U11 IS31FL3739-GRLS4-TR, U2 TLC555CDR, U3 SN74HC08DR, U4 SN74HC08DR, U6 SN74HC08DR, U7 SN74HC08DR, U8 BNO055

Commit message: Add level shifters to leg board, re-route and export
Parts:
- added U10, U12, U13, U14, U5, U9: 74HCT125D, LevelShifter:74HCT125D, symbol LevelShifter:74HCT125D
- J1, J10, J11, J12, J13, J14, J15, J16, J17, J18, J19, J20, J6, J7, J8, J9: now left out of the parts list
Connections:
- net +3.3V: no longer J10.2 (Pin_2), J11.2 (Pin_2), J12.2 (Pin_2), J13.2 (Pin_2), J6.2 (Pin_2), J7.2 (Pin_2), J8.2 (Pin_2), J9.2 (Pin_2)
- net GND: now also U10.1 (1OE*), U10.10 (3OE*), U10.13 (4OE*), U10.4 (2OE*), U10.7 (GND), U12.1 (1OE*), U12.10 (3OE*), U12.13 (4OE*), U12.4 (2OE*), U12.7 (GND), U13.1 (1OE*), U13.10 (3OE*), U13.13 (4OE*), U13.4 (2OE*), U13.7 (GND), U14.1 (1OE*), U14.10 (3OE*), U14.13 (4OE*), U14.4 (2OE*), U14.7 (GND), U5.1 (1OE*), U5.10 (3OE*), U5.13 (4OE*), U5.4 (2OE*), U5.7 (GND), U9.1 (1OE*), U9.10 (3OE*), U9.13 (4OE*), U9.4 (2OE*), U9.7 (GND)
- net LPWM1: now also U5.5 (2A*); no longer J6.7 (Pin_7)
- net LPWM2: now also U5.12 (4A); no longer J7.7 (Pin_7)
- net LPWM3: now also U9.5 (2A*); no longer J8.7 (Pin_7)
- net LPWM4: now also U9.12 (4A); no longer J9.7 (Pin_7)
- net LPWM5: now also U10.5 (2A*); no longer J10.7 (Pin_7)
- net LPWM6: now also U10.9 (3A); no longer J11.7 (Pin_7)
- net LPWM7: now also U12.5 (2A*); no longer J12.7 (Pin_7)
- net LPWM8: now also U12.9 (3A); no longer J13.7 (Pin_7)
- net PWMEN1: now also U13.2 (1A); no longer J6.5 (Pin_5), J6.6 (Pin_6)
- net PWMEN2: now also U13.5 (2A*); no longer J7.5 (Pin_5), J7.6 (Pin_6)
- net PWMEN3: now also U13.12 (4A); no longer J8.5 (Pin_5), J8.6 (Pin_6)
- net PWMEN4: now also U13.9 (3A); no longer J9.5 (Pin_5), J9.6 (Pin_6)
- net PWMEN5: now also U14.2 (1A); no longer J10.5 (Pin_5), J10.6 (Pin_6)
- net PWMEN6: now also U14.5 (2A*); no longer J11.5 (Pin_5), J11.6 (Pin_6)
- net PWMEN7: now also U14.9 (3A); no longer J12.5 (Pin_5), J12.6 (Pin_6)
- net PWMEN8: now also U14.12 (4A); no longer J13.5 (Pin_5), J13.6 (Pin_6)
- net RPWM1: now also U5.2 (1A); no longer J6.8 (Pin_8)
- net RPWM2: now also U5.9 (3A); no longer J7.8 (Pin_8)
- net RPWM3: now also U9.2 (1A); no longer J8.8 (Pin_8)
- net RPWM4: now also U9.9 (3A); no longer J9.8 (Pin_8)
- net RPWM5: now also U10.2 (1A); no longer J10.8 (Pin_8)
- net RPWM6: now also U10.12 (4A); no longer J11.8 (Pin_8)
- net RPWM7: now also U12.2 (1A); no longer J12.8 (Pin_8)
- net RPWM8: now also U12.12 (4A); no longer J13.8 (Pin_8)
- net +5V: now reaches U1.49 (VUSB)
- net +5V: now also J10.2 (Pin_2), J11.2 (Pin_2), J12.2 (Pin_2), J13.2 (Pin_2), J6.2 (Pin_2), J7.2 (Pin_2), J8.2 (Pin_2), J9.2 (Pin_2), U10.14 (VCC), U12.14 (VCC), U13.14 (VCC), U14.14 (VCC), U5.14 (VCC), U9.14 (VCC)
- new net LPWM1_5V: J6.7 (Pin_7), U5.6 (2Y)
- new net LPWM2_5V: J7.7 (Pin_7), U5.11 (4Y)
- new net LPWM3_5V: J8.7 (Pin_7), U9.6 (2Y)
- new net LPWM4_5V: J9.7 (Pin_7), U9.11 (4Y)
- new net LPWM5_5V: J10.7 (Pin_7), U10.6 (2Y)
- new net LPWM6_5V: J11.7 (Pin_7), U10.8 (3Y)
- new net LPWM7_5V: J12.7 (Pin_7), U12.6 (2Y)
- new net LPWM8_5V: J13.7 (Pin_7), U12.8 (3Y)
- new net PWMEN1_5V: J6.5 (Pin_5), J6.6 (Pin_6), U13.3 (1Y)
- new net PWMEN2_5V: J7.5 (Pin_5), J7.6 (Pin_6), U13.6 (2Y)
- new net PWMEN3_5V: J8.5 (Pin_5), J8.6 (Pin_6), U13.11 (4Y)
- new net PWMEN4_5V: J9.5 (Pin_5), J9.6 (Pin_6), U13.8 (3Y)
- new net PWMEN5_5V: J10.5 (Pin_5), J10.6 (Pin_6), U14.3 (1Y)
- new net PWMEN6_5V: J11.5 (Pin_5), J11.6 (Pin_6), U14.6 (2Y)
- new net PWMEN7_5V: J12.5 (Pin_5), J12.6 (Pin_6), U14.8 (3Y)
- new net PWMEN8_5V: J13.5 (Pin_5), J13.6 (Pin_6), U14.11 (4Y)
- new net RPWM1_5V: J6.8 (Pin_8), U5.3 (1Y)
- new net RPWM2_5V: J7.8 (Pin_8), U5.8 (3Y)
- new net RPWM3-5V: U9.3 (1Y)
- new net RPWM3_5V: J8.8 (Pin_8)
- new net RPWM4_5V: J9.8 (Pin_8), U9.8 (3Y)
- new net RPWM5_5V: J10.8 (Pin_8), U10.3 (1Y)
- new net RPWM6_5V: J11.8 (Pin_8), U10.11 (4Y)
- new net RPWM7_5V: J12.8 (Pin_8), U12.3 (1Y)
- new net RPWM8_5V: J13.8 (Pin_8), U12.11 (4Y)
Other:
- note added: "3.3V to 5V LEVEL SHIFTERS"
- note added: "PWM ENABLED 1-4"
- note added: "PWM ENABLED 5-8"
- note added: "PWM1"
- note added: "PWM2"
- note added: "PWM3"
- note added: "PWM4"
- note added: "PWM5"
- note added: "PWM6"
- note added: "PWM7"
- note added: "PWM8"
- moved on the sheet: C1, C10, C2, C3, C4, C5, C6, C7, C8, C9, D1, D10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
