File: boards/LegRobotBoardTeensy/LegRobotBoardTeensy.kicad_pcb (KiCad board)
At the start: 2 copper layers, 178.2 x 110.9 mm, 175 parts, among them J1 IDC, J10 IDC, J11 IDC, J12 IDC, J13 IDC, J14 IDC, J15 IDC, J16 IDC, J17 Conn_01x10, J18 Conn_01x10, J19 Conn_01x10, J2 B3B-XH-A, J20 Conn_01x10, J3 B3B-XH-A, J4 B3B-XH-A, J5 B3B-XH-A, J6 IDC, J7 IDC, J8 IDC, J9 IDC, Q1 AO3400A, Q10 AO3400A, Q11 AO3400A, Q12 AO3400A, Q13 AO3400A, Q14 AO3400A, Q15 AO3400A, Q16 AO3400A, Q17 AO3400A, Q18 AO3400A, Q19 AO3400A, Q2 AO3400A, Q20 AO3400A, Q21 AO3400A, Q22 AO3400A, Q23 AO3400A, Q24 AO3400A, Q3 AO3400A, Q4 AO3400A, Q5 AO3400A, Q6 AO3400A, Q7 AO3400A, Q8 AO3400A, Q9 AO3400A, U1 Teensy4.0, U11 IS31FL3739-GRLS4-TR, U2 TLC555CDR, U3 SN74HC08DR, U4 SN74HC08DR, U5 PCA9685PW_118, U6 SN74HC08DR, U7 SN74HC08DR, U8 BNO055

Commit message: Pre-flight main board
Changed lines of the file:
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@@
 	(gr_poly
 		(pts
-			(xy 235.494187 92.913285) (xy 232.244606 90.453981) (xy 235.494187 87.994842) (xy 236.091154 87.994842)
-			(xy 236.091154 92.913285)
-		)
-		(stroke
-			(width 0.330729)
-			(type solid)
-			(color 255 255 255 1)
-		)
-		(fill no)
-		(layer "F.SilkS")
-	)
-	(gr_poly
-		(pts
 			(xy 143.969561 35.755493) (xy 144.274956 35.77471) (xy 144.574925 35.806407) (xy 144.868925 35.850313)
 			(xy 145.156414 35.906156) (xy 145.436849 35.973665) (xy 145.709688 36.052568) (xy 145.974387 36.142595)
@@
 	(gr_poly
 		(pts
-			(xy 231.665813 89.87527) (xy 231.068846 89.87527) (xy 231.068846 84.956993) (xy 231.665813 84.956993)
-			(xy 234.915394 87.416131)
-		)
-		(stroke
-			(width 0.330729)
-			(type solid)
-			(color 255 255 255 1)
-		)
-		(fill no)
-		(layer "F.SilkS")
-	)
-	(gr_poly
-		(pts
 			(xy 122.915948 37.971527) (xy 113.285114 37.971527) (xy 123.471572 48.157985) (xy 121.989906 49.824859)
 			(xy 111.803447 39.638402) (xy 111.803447 49.269236) (xy 109.395739 49.269236) (xy 109.395739 35.749027)
@@
 	(gr_poly
 		(pts
-			(xy 76.154187 84.956993) (xy 76.751154 84.956993) (xy 76.751154 89.87527) (xy 76.154187 89.87527)
-			(xy 72.904606 87.416131)
-		)
-		(stroke
-			(width 0.330729)
-			(type solid)
-			(color 255 255 255 1)
-		)
-		(fill no)
-		(layer "F.SilkS")
-	)
-	(gr_poly
-		(pts
 			(xy 237.454019 51.375228) (xy 237.46183 51.375822) (xy 237.469527 51.3768) (xy 237.4771 51.378152)
 			(xy 237.484541 51.379869) (xy 237.491839 51.381941) (xy 237.498985 51.384359) (xy 237.505969 51.387113)
@@
 	(gr_poly
 		(pts
-			(xy 235.494187 98.98923) (xy 232.244606 96.529927) (xy 235.494187 94.070787) (xy 236.091154 94.070787)
-			(xy 236.091154 98.98923)
-		)
-		(stroke
-			(width 0.330729)
-			(type solid)
-			(color 255 255 255 1)
-		)
-		(fill no)
-		(layer "F.SilkS")
-	)
-	(gr_poly
-		(pts
 			(xy 79.642333 56.005417) (xy 79.650143 56.006011) (xy 79.65784 56.006989) (xy 79.665414 56.008341)
 			(xy 79.672855 56.010059) (xy 79.680153 56.012131) (xy 79.687299 56.014549) (xy 79.694283 56.017302)
@@
 	(gr_poly
 		(pts
-			(xy 76.154187 97.108785) (xy 76.751154 97.108785) (xy 76.751154 102.027227) (xy 76.154187 102.027227)
-			(xy 72.904606 99.567924)
-		)
-		(stroke
-			(width 0.330729)
-			(type solid)
-			(color 255 255 255 1)
-		)
-		(fill no)
-		(layer "F.SilkS")
-	)
-	(gr_poly
-		(pts
 			(xy 79.642333 53.690334) (xy 79.650143 53.690927) (xy 79.65784 53.691905) (xy 79.665414 53.693258)
 			(xy 79.672855 53.694975) (xy 79.680153 53.697047) (xy 79.687299 53.699465) (xy 79.694283 53.702219)
@@
 	(gr_poly
 		(pts
-			(xy 72.325813 100.146715) (xy 75.575394 102.606019) (xy 72.325813 105.065158) (xy 71.728846 105.065158)
-			(xy 71.728846 100.146715)
-		)
-		(stroke
-			(width 0.330729)
-			(type solid)
-			(color 255 255 255 1)
-		)
-		(fill no)
-		(layer "F.SilkS")
-	)
-	(gr_poly
-		(pts
 			(xy 72.696959 53.690306) (xy 72.70477 53.6909) (xy 72.712468 53.691877) (xy 72.720043 53.69323) (xy 72.727485 53.694947)
 			(xy 72.734784 53.697019) (xy 72.741932 53.699437) (xy 72.748918 53.702191) (xy 72.755732 53.705271)
@@
 	(gr_poly
 		(pts
-			(xy 231.665813 102.027176) (xy 231.068846 102.027176) (xy 231.068846 97.108899) (xy 231.665813 97.108899)
-			(xy 234.915394 99.568038)
-		)
-		(stroke
-			(width 0.330729)
-			(type solid)
-			(color 255 255 255 1)
-		)
-		(fill no)
-		(layer "F.SilkS")
-	)
-	(gr_poly
-		(pts
 			(xy 228.193552 60.635629) (xy 228.201363 60.636223) (xy 228.209061 60.637202) (xy 228.216635 60.638555)
 			(xy 228.224077 60.640274) (xy 228.231377 60.642347) (xy 228.238524 60.644767) (xy 228.24551 60.647522)
@@
 	(gr_poly
 		(pts
-			(xy 235.494187 105.065093) (xy 232.244606 102.605953) (xy 235.494187 100.146815) (xy 236.091154 100.146815)
-			(xy 236.091154 105.065093)
-		)
-		(stroke
-			(width 0.330729)
-			(type solid)
-			(color 255 255 255 1)
-		)
-		(fill no)
-		(layer "F.SilkS")
-	)
-	(gr_poly
-		(pts
 			(xy 101.035908 35.757709) (xy 101.375713 35.783754) (xy 101.709549 35.827162) (xy 102.036603 35.887933)
 			(xy 102.35606 35.966068) (xy 102.667107 36.061566) (xy 102.968929 36.174427) (xy 103.260714 36.304652)
@@
 	(gr_poly
 		(pts
-			(xy 72.325813 87.994907) (xy 75.575394 90.454047) (xy 72.325813 92.913185) (xy 71.728846 92.913185)
-			(xy 71.728846 87.994907)
-		)
-		(stroke
-			(width 0.330729)
-			(type solid)
-			(color 255 255 255 1)
-		)
-		(fill no)
-		(layer "F.SilkS")
-	)
-	(gr_poly
-		(pts
 			(xy 68.066759 56.005417) (xy 68.07457 56.006011) (xy 68.082268 56.006989) (xy 68.089842 56.008341)
 			(xy 68.097284 56.010059) (xy 68.104584 56.012131) (xy 68.111731 56.014549) (xy 68.118717 56.017302)
@@
 	(gr_poly
 		(pts
-			(xy 76.154187 91.032824) (xy 76.751154 91.032824) (xy 76.751154 95.951101) (xy 76.154187 95.951101)
-			(xy 72.904606 93.491962)
-		)
-		(stroke
-			(width 0.330729)
-			(type solid)
-			(color 255 255 255 1)
-		)
-		(fill no)
-		(layer "F.SilkS")
-	)
-	(gr_poly
-		(pts
 			(xy 117.35014 99.861571) (xy 117.357343 99.86203) (xy 117.364382 99.86279) (xy 117.371251 99.863845)
 			(xy 117.377945 99.865191) (xy 117.384461 99.866823) (xy 117.390792 99.868736) (xy 117.396934 99.870925)
@@
 	(gr_poly
 		(pts
-			(xy 231.665813 108.103007) (xy 231.068846 108.103007) (xy 231.068846 103.18473) (xy 231.665813 103.18473)
-			(xy 234.915394 105.643869)
-		)
-		(stroke
-			(width 0.330729)
-			(type solid)
-			(color 255 255 255 1)
-		)
-		(fill no)
-		(layer "F.SilkS")
-	)
-	(gr_poly
-		(pts
 			(xy 189.730029 99.861571) (xy 189.737232 99.86203) (xy 189.744271 99.86279) (xy 189.75114 99.863845)
 			(xy 189.757834 99.865191) (xy 189.76435 99.866823) (xy 189.770681 99.868736) (xy 189.776823 99.870925)
@@
 	(gr_poly
 		(pts
-			(xy 231.665813 95.951215) (xy 231.068846 95.951215) (xy 231.068846 91.032773) (xy 231.665813 91.032773)
-			(xy 234.915394 93.492076)
-		)
-		(stroke
-			(width 0.330729)
-			(type solid)
-			(color 255 255 255 1)
-		)
-		(fill no)
-		(layer "F.SilkS")
-	)
-	(gr_poly
-		(pts
 			(xy 232.823752 60.635629) (xy 232.831563 60.636223) (xy 232.839261 60.637202) (xy 232.846836 60.638555)
 			(xy 232.854278 60.640274) (xy 232.861577 60.642347) (xy 232.868725 60.644767) (xy 232.875711 60.647522)
@@
 	(gr_poly
 		(pts
-			(xy 72.325813 94.07077) (xy 75.575394 96.530073) (xy 72.325813 98.989213) (xy 71.728846 98.989213)
-			(xy 71.728846 94.07077)
-		)
-		(stroke
-			(width 0.330729)
-			(type solid)
-			(color 255 255 255 1)
-		)
-		(fill no)
-		(layer "F.SilkS")
-	)
-	(gr_poly
-		(pts
 			(xy 220.030744 98.196592) (xy 220.085287 98.201578) (xy 220.138213 98.209752) (xy 220.189564 98.221002)
 			(xy 220.239384 98.235217) (xy 220.287717 98.252286) (xy 220.334606 98.272096) (xy 220.380095 98.294537)
@@
 	(gr_poly
 		(pts
-			(xy 76.154187 103.18473) (xy 76.751154 103.18473) (xy 76.751154 108.103007) (xy 76.154187 108.103007)
-			(xy 72.904606 105.643869)
-		)
-		(stroke
-			(width 0.330729)
-			(type solid)
-			(color 255 255 255 1)
-		)
-		(fill no)
-		(layer "F.SilkS")
-	)
-	(gr_poly
-		(pts
 			(xy 159.216776 49.269236) (xy 156.80907 49.269236) (xy 156.80907 39.638402) (xy 152.919696 44.083403)
 			(xy 149.956357 44.083403) (xy 157.179486 35.749027) (xy 159.216776 35.749027)
@@
 	)
 	(group ""
-		(members "0031d323-2b6b-439d-b327-e77e99ef24ec" "1e12d83f-ab1b-4354-90aa-7a45f1db8419"
-			"36418407-8df9-49ec-ae44-3dec7df0693b" "796bd5fc-db61-44d6-9c6d-afd1f469cbbc"
-			"8616f52e-ad49-4b8c-ab90-523d1fc25b46" "be094907-fb75-4566-bb38-f1a7d1d769fd"
-			"c47fe27a-dbaf-46e2-877a-a4acb4c7db01"
-		)
-	)
-	(group ""
 		(members "8130a495-d03c-4b6a-99d3-b76ee8ec899a" "82b7f386-41f9-4b44-8e41-28e1fa265e30")
 	)
@@
 	)
 	(group ""
-		(members "2b8170ee-6588-462c-a845-67b4caf334c4" "400acf30-b1e7-4714-97fd-5102793b9e33"
-			"5e735bef-2616-4c0e-9193-fe280d0b852b" "90d82b74-eea9-455d-a8eb-00988a93cacc"
-			"b538e87f-8b93-44a3-a83f-027f70cfc1b0" "e94f83e4-44bd-442d-8604-f2696e34401a"
-			"f6a8ba1b-29ff-4c35-b4d7-5e05bcfe7f79"
-		)
-	)
-	(group ""

Commit message: Re-finalize leg board
Parts:
- removed R27: 10K, CRCW060310K0FKEA:CRCW060310K0FKEA
- removed U5: PCA9685PW_118, PCA9685PW,118:PCA9685PW,118
- D1, D2, D3, D4, D5, D6, D7, D8: footprint NCD0603R1:NCD0603R1 -> XL-1608SURC-06:XL-1608SURC-06
- J17, J18, J19, J20: footprint DIP:DIP-10_W15.24mm -> Package_DIP:DIP-10_W10.16mm
- R10, R3, R4, R5, R6, R7, R8, R9: value 1K -> 470R; footprint RCG06031K00FKEA:RCG06031K00FKEA -> RC0603FR-07470RL:RC0603FR-07470RL
- U1: value Teensy4.0 -> Teensy4.1; footprint Teensy40:Teensy40 -> Teensy4.1:Teensy41
- moved R83 85.8 mm to (225.7, 95.3)
- moved C9 85.3 mm to (226.4, 89.6)
- moved R84 84.8 mm to (225.7, 92.6)
- moved U11 81.3 mm to (233.5, 93.3)
- moved C10 79.6 mm to (223.8, 89.6)
- moved R82 78.7 mm to (222.4, 92.7)
- moved R79 78.6 mm to (222.3, 95.3)
- moved C1 12.7 mm to (148.1, 76.7)
- moved C2 12.7 mm to (159.8, 81.0)
- moved C4 12.7 mm to (153.6, 74.2)
- moved R1 12.7 mm to (160.3, 78.6)
- moved R2 12.7 mm to (160.3, 76.0)
- moved U2 12.7 mm to (153.8, 78.2)
- moved U1 12.6 mm to (153.9, 114.1)
- moved J17 6.84 mm to (70.6, 73.8)
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Connections:
- J17 pad 1: DIGIT_C -> DIGIT_G
- J17 pad 10: DIGIT_A -> COM0
- J17 pad 3: DIGIT_E -> DIGIT_A
- J17 pad 4: DIGIT_D -> DIGIT_F
- J17 pad 5: DIGIT_G -> COM1
- J17 pad 6: DIGIT_F -> DIGIT_D
- J17 pad 7: COM1 -> DIGIT_E
- J17 pad 8: COM0 -> DIGIT_C
- J18 pad 1: DIGIT_C -> DIGIT_G
- J18 pad 10: DIGIT_A -> COM2
- J18 pad 3: DIGIT_E -> DIGIT_A
- J18 pad 4: DIGIT_D -> DIGIT_F
- J18 pad 5: DIGIT_G -> COM3
- J18 pad 6: DIGIT_F -> DIGIT_D
- J18 pad 7: COM3 -> DIGIT_E
- J18 pad 8: COM2 -> DIGIT_C
- J19 pad 1: DIGIT_C -> DIGIT_G
- J19 pad 10: DIGIT_A -> COM4
- J19 pad 3: DIGIT_E -> DIGIT_A
- J19 pad 4: DIGIT_D -> DIGIT_F
- J19 pad 5: DIGIT_G -> COM5
- J19 pad 6: DIGIT_F -> DIGIT_D
- J19 pad 7: COM5 -> DIGIT_E
- J19 pad 8: COM4 -> DIGIT_C
- J20 pad 1: DIGIT_C -> DIGIT_G
- J20 pad 10: DIGIT_A -> COM6
- J20 pad 3: DIGIT_E -> DIGIT_A
- J20 pad 4: DIGIT_D -> DIGIT_F
- J20 pad 5: DIGIT_G -> COM7
- J20 pad 6: DIGIT_F -> DIGIT_D
- J20 pad 7: COM7 -> DIGIT_E
- J20 pad 8: COM6 -> DIGIT_C
- R29 pad 2: A0 -> POT1
- R30 pad 2: A1 -> POT2
- R31 pad 2: A2 -> POT3
- R32 pad 2: A3 -> POT4
- U1 pad 10: ENCODER4_B -> RPWM5
- U1 pad 11: PWMEN2 -> LPWM5
- U1 pad 12: PWMEN3 -> RPWM6
- U1 pad 13: PWMEN4 -> LPWM6
- U1 pad 14: PWMEN5 -> RPWM7
- U1 pad 15: unconnected-(U1-VBAT-Pad15) -> +3.3V
- U1 pad 16: +3.3V -> ENCODER3_I
- U1 pad 17: GND -> ENCODER4_I
- U1 pad 18: unconnected-(U1-PROGRAM-Pad18) -> PWMEN1
- U1 pad 19: unconnected-(U1-ON_OFF-Pad19) -> PWMEN2
- U1 pad 2: ENCODER1_A -> RPWM1
- U1 pad 20: PWMEN6 -> PWMEN3
- U1 pad 21: A0 -> PWMEN4
- U1 pad 22: A1 -> PWMEN5
- U1 pad 23: A2 -> PWMEN6
- U1 pad 24: A3 -> ENCODER1_A
- U1 pad 25: SDA -> ENCODER1_B
- U1 pad 26: SCL -> ENCODER2_A
- U1 pad 27: PWMEN7 -> ENCODER2_B
- U1 pad 28: PWMEN8 -> ENCODER3_A
- U1 pad 29: ENCODER1_I -> ENCODER3_B
- U1 pad 3: ENCODER1_B -> LPWM1
- U1 pad 30: ENCODER2_I -> ENCODER4_A
- U1 pad 31: unconnected-(U1-3V3-Pad31) -> ENCODER4_B
- U1 pad 32: unconnected-(U1-GND-Pad32) -> POT1
- U1 pad 33: unconnected-(U1-VIN-Pad33) -> POT2
- U1 pad 34: unconnected-(U1-VUSB-Pad34) -> GND
- U1 pad 35: ENCODER3_I -> LPWM7
- U1 pad 36: ENCODER4_I -> RPWM8
- U1 pad 37: unconnected-(U1-26_A12_MOSI1-Pad37) -> LPWM8
- U1 pad 38: unconnected-(U1-27_A13_SCK1-Pad38) -> POT3
- U1 pad 39: unconnected-(U1-28_RX7-Pad39) -> POT4
- U1 pad 4: ENCODER2_A -> RPWM2
- U1 pad 40: unconnected-(U1-29_TX7-Pad40) -> SDA
- U1 pad 41: unconnected-(U1-30_CRX3-Pad41) -> SCL
- U1 pad 42: unconnected-(U1-31_CTX3-Pad42) -> PWMEN7
- U1 pad 43: unconnected-(U1-32_OUT1B-Pad43) -> PWMEN8
- U1 pad 44: unconnected-(U1-33_MCLK2-Pad44) -> ENCODER1_I
- U1 pad 5: ENCODER2_B -> LPWM2
- U1 pad 6: ENCODER3_A -> RPWM3
- U1 pad 7: ENCODER3_B -> LPWM3
- U1 pad 8: PWMEN1 -> RPWM4
- U1 pad 9: ENCODER4_A -> LPWM4
Routing:
- net A1: track 137.4 -> 0.00 mm, vias 1 -> 0
- net SDA: track 77.1 -> 201.2 mm, vias 4 -> 5
- net POT2: track 0.00 -> 120.3 mm, vias 0 -> 1
- net COM1: track 79.3 -> 199.3 mm, vias 0 -> 3
- net COM0: track 78.2 -> 193.9 mm, vias 0 -> 2
- net COM5: track 147.9 -> 261.4 mm, vias 4 -> 3
- net COM2: track 141.3 -> 31.6 mm, vias 3 -> 1
- net COM7: track 128.3 -> 30.7 mm, vias 4 -> 1
- net A0: track 92.8 -> 0.00 mm, vias 2 -> 0
- net COM6: track 118.1 -> 27.6 mm, vias 4 -> 1
- net SCL: track 76.5 -> 164.2 mm, vias 2 -> 3
- net A3: track 83.5 -> 0.00 mm, vias 2 -> 0
- net POT1: track 0.00 -> 81.0 mm, vias 0 -> 2
- net +3.3V: track 752.4 -> 831.1 mm
- net DIGIT_G: track 349.3 -> 272.5 mm, vias 3 -> 5
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Other:
- board text added: "01binary"
- board text added: "tech art"
- board text removed: "C2"
- board text removed: "C3"
- board text removed: "C4"
- board text removed: "C5"
- board text removed: "C6"
- board text removed: "C7"
