File: boards/ArmEncoderBoard/ArmEncoderBoard.kicad_pcb (KiCad board)
At the start: 2 copper layers, 34 x 34 mm, 25 parts, among them J1 Conn_01x05, Q1 SS8050, Q2 SS8050, U1 DBV6, U2 AS5045B

Commit message: Pre-flight on two encoder boards
Parts:
- C2: value 0.1uF -> 100nF
- U1: value DBV6 -> SN74LVC2G17DBVR
- moved R3 3.54 mm to (129.1, 84.0)
- moved R4 3.47 mm to (148.3, 84.2)
- moved D2 0.17 mm to (148.3, 82.2)
Routing:
- net VIN: track 47.7 -> 42.6 mm
- net /BLUE_ANODE: track 4.09 -> 2.35 mm
- net /RED_ANODE: track 4.25 -> 2.59 mm
- net /BLUE_CATHODE: track 14.2 -> 13.7 mm
Changed lines of the file:
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@@
 	(footprint "LedBlue:YLED0603B"
 		(layer "F.Cu")
-		(at 129.05 82.2)
+		(at 129.05 82.181575)
 		(property "Reference" "D1"
-			(at 0 1.548625 0)
+			(at -2.1 0.018425 0)
 			(unlocked yes)
 			(layer "F.SilkS")
@@
 		)
 		(pad "1" smd rect
-			(at -0.6223 -0.001375)
+			(at 0.6223 -0.001375)
 			(size 0.762 0.8636)
 			(layers "F.Cu" "F.Mask" "F.Paste")
@@
 		)
 		(pad "2" smd rect
-			(at 0.6223 -0.001375)
+			(at -0.6223 -0.001375)
 			(size 0.762 0.8636)
 			(layers "F.Cu" "F.Mask" "F.Paste")
@@
 			(polygon
 				(pts
-					(xy 128.8595 81.792225) (xy 129.2405 81.792225) (xy 129.2405 82.605025) (xy 128.8595 82.605025)
+					(xy 128.8595 81.7738) (xy 129.2405 81.7738) (xy 129.2405 82.5866) (xy 128.8595 82.5866)
 				)
 			)
 		)
 		(group ""
-			(members "0100014e-db4a-472f-9bde-102add28c4d1" "025f57e7-6d5f-4346-989f-b10fb728b310"
-				"5e8504f6-3a37-4747-b3ff-e2ac54052047" "eb10f852-7608-4674-a56f-17776146af03"
+			(members "2fce0801-b599-416b-9a28-ec66d2f29070" "4c2caeea-5ffc-4bf9-a038-e9676119c98e"
+				"cb6d4ac6-8f4b-4a35-be16-be7872730078" "e2259e4a-c0e1-4dee-9810-fc8781127cd8"
 			)
 		)
@@
 			)
 		)
-		(property "Value" "DBV6"
+		(property "Value" "SN74LVC2G17DBVR"
 			(at 0 0 0)
 			(unlocked yes)
@@
 	(footprint "LedRed:YLED0603R"
 		(layer "F.Cu")
-		(at 148.1777 82.1986)
+		(at 148.35 82.1802)
 		(property "Reference" "D2"
-			(at -0.0277 1.65 0)
+			(at 2.35 0.0198 0)
 			(unlocked yes)
 			(layer "F.SilkS")
@@
 		)
 		(pad "1" smd rect
-			(at -0.6223 0)
+			(at 0.6223 0)
 			(size 0.762 0.8636)
 			(layers "F.Cu" "F.Mask" "F.Paste")
@@
 		)
 		(pad "2" smd rect
-			(at 0.6223 0)
+			(at -0.6223 0)
 			(size 0.762 0.8636)
 			(layers "F.Cu" "F.Mask" "F.Paste")
@@
 			(polygon
 				(pts
-					(xy 147.9872 81.7922) (xy 148.3682 81.7922) (xy 148.3682 82.605) (xy 147.9872 82.605)
+					(xy 148.1595 81.7738) (xy 148.5405 81.7738) (xy 148.5405 82.5866) (xy 148.1595 82.5866)
 				)
 			)
 		)
 		(group ""
-			(members "05b01988-7c54-4fe5-954b-3361d50654ac" "066d1c90-1073-44ed-8cdd-aea4cde48923"
-				"1c348134-b67e-48aa-9ebe-9242fb27f465" "26292bf5-9d36-4f02-930b-19808e1ac686"
-				"32d1b891-ecb0-46a0-9e4c-83ff73103c07" "38275ea2-9ee2-469e-9cd3-a6f9244b07d9"
-				"3b6ecf8d-6916-4bf6-8bfb-9b2024dfe9ff" "3e34ce83-d91b-4210-bc91-a77855c5565a"
-				"6cdd37fc-c30d-4ee3-aab1-f7aae5a0a799" "78a3e141-e400-4ac9-813b-f4bd467607f6"
-				"7c4178ac-632a-4fe4-8522-e90f0ae094cc" "8feb024c-b0fe-4d03-a796-62247da453bb"
-				"c74250a4-f3e0-4304-877d-e74fb513f51e" "c823b551-ced1-4a09-9d0b-f473d22536e8"
-				"ca66b30e-a4b5-4ff5-a9ea-ef687d6a75e2" "d8e02e98-af3a-4b91-a43e-a0289d4b1f63"
-				"f3493101-4c6b-4fe1-8823-61cbbbaf49a1" "f6326e0d-0cb9-4f98-a252-c0b4dda1dc5a"
-				"fe62e95f-afb2-478e-be7f-488f7e700c41"
-			)
-		)
-		(group ""
-			(members "0b28b877-760a-4570-963d-161da1ecbe3c" "3ca774cc-c1b5-414a-ad66-6c2a10f970c3"
-				"88fd0d4b-5c7f-45bc-b7a4-b9486859a690" "df297313-ca28-47bd-9903-51e7eabaa262"
+			(members "2838feab-9907-4163-b272-768ffd1597eb" "37a75fa1-47a7-4eb8-887b-f1942aa10586"
+				"631b936f-8bc4-49c3-b1d9-cb89c1ea0fef" "9073877d-4c01-4eb4-b25a-0fa23aeda077"
 			)
 		)
@@
 		(sheetname "/")
 		(sheetfile "ArmEncoderBoard.kicad_sch")
-		(attr through_hole exclude_from_pos_files exclude_from_bom)
+		(attr through_hole exclude_from_pos_files exclude_from_bom dnp)
 		(fp_line
 			(start -2.85 -2.75)
@@
 		(tags "CC0603KRX7R9BB104 ")
 		(property "Reference" "C2"
-			(at 0.0223 -1.15 0)
+			(at 0.0223 1.6 0)
 			(unlocked yes)
 			(layer "F.SilkS")
@@
 			)
 		)
-		(property "Value" "0.1uF"
+		(property "Value" "100nF"
 			(at 0 0 0)
 			(unlocked yes)
@@
 	(footprint "Resistor150:RESC1607X60N"
 		(layer "F.Cu")
-		(at 125.915 82.3486)
+		(at 129.05 83.9938)
 		(property "Reference" "R3"
-			(at 0.035 1.45 0)
+			(at -2.1 0.0062 0)
 			(layer "F.SilkS")
 			(effects
@@
 			(polygon
 				(pts
-					(xy 125.5721 81.993) (xy 126.2579 81.993) (xy 126.2579 82.7042) (xy 125.5721 82.7042)
+					(xy 128.7071 83.6382) (xy 129.3929 83.6382) (xy 129.3929 84.3494) (xy 128.7071 84.3494)
 				)
 			)
@@
 	(footprint "Resistor1K:RCG06031K00FKEA"
 		(layer "F.Cu")
-		(at 151.285 82.3486)
+		(at 148.35 84.2)
 		(property "Reference" "R4"
-			(at -0.035 1.5 0)
+			(at 2.35 0 0)
 			(layer "F.SilkS")
 			(effects
@@
 			)
 		)
+		(property "LCSC" "C81464"
+			(at 0 0 90)
+			(unlocked yes)
+			(layer "F.Fab")
+			(hide yes)
+			(effects
+				(font
+					(size 1 1)
+					(thickness 0.15)
+				)
+			)
+		)
 		(property ki_fp_filters "SOT?23*")
 		(sheetname "/")
@@
 			)
 		)
+		(property "LCSC" "C105579"
+			(at 0 0 0)
+			(unlocked yes)
+			(layer "F.Fab")
+			(hide yes)
+			(effects
+				(font
+					(size 1 1)
+					(thickness 0.15)
+				)
+			)
+		)
 		(property ki_fp_filters "R_*")
 		(sheetname "/")
@@
 	)
 	(segment
-		(start 149.7633 82.3486)
-		(end 149.7633 82.5769)
+		(start 145.4985 81.4288)
+		(end 144.348 81.4288)
 		(width 0.25)
 		(layer "F.Cu")
@@
 	)
 	(segment
-		(start 145.4985 81.4288)
-		(end 144.348 81.4288)
+		(start 133.8 84.1818)
+		(end 133.7483 84.1818)
 		(width 0.25)
 		(layer "F.Cu")
@@
 	)
 	(segment
-		(start 149.3831 82.9571)
-		(end 146.9379 82.9571)
+		(start 133.8 84.917)
+		(end 133.8 84.1818)
 		(width 0.25)
 		(layer "F.Cu")
@@
 	)
 	(segment
-		(start 133.8 84.1818)
-		(end 133.7483 84.1818)
+		(start 139.4361 77.7668)
+		(end 141.4443 79.775)
 		(width 0.25)
 		(layer "F.Cu")
@@
 	)
 	(segment
-		(start 133.8 84.917)
-		(end 133.8 84.1818)
+		(start 128.3769 83.9938)
+		(end 128.3769 84.6248)
 		(width 0.25)
 		(layer "F.Cu")
@@
 	)
 	(segment
-		(start 139.4361 77.7668)
-		(end 141.4443 79.775)
+		(start 147.585 84.2)
+		(end 147.4985 84.2)
 		(width 0.25)
 		(layer "F.Cu")
@@
 	)
 	(segment
-		(start 145.4985 82.2)
-		(end 146.1808 82.2)
+		(start 128.3769 84.6248)
+		(end 128.6691 84.917)
 		(width 0.25)
 		(layer "F.Cu")
@@
 	)
 	(segment
-		(start 132.8223 83.4256)
-		(end 125.6112 83.4256)
-		(width 0.25)
-		(layer "F.Cu")
-		(net 4)
-	)
-	(segment
 		(start 141.4443 79.775)
 		(end 142.1375 79.775)
@@
 	)
 	(segment
-		(start 149.7633 82.5769)
-		(end 149.3831 82.9571)
-		(width 0.25)
-		(layer "F.Cu")
-		(net 4)
-	)
-	(segment
 		(start 140.9163 80.425)
 		(end 136.4243 84.917)
@@
 	)
 	(segment
-		(start 146.9379 82.9571)
-		(end 146.1808 82.2)
+		(start 128.6691 84.917)
+		(end 133.8 84.917)
 		(width 0.25)
 		(layer "F.Cu")
@@
 	)
 	(segment
-		(start 125.2419 82.3486)
-		(end 125.2419 83.0563)
-		(width 0.25)
-		(layer "F.Cu")
-		(net 4)
-	)
-	(segment
-		(start 150.52 82.3486)
-		(end 149.7633 82.3486)
+		(start 147.4985 84.2)
+		(end 145.4985 82.2)
 		(width 0.25)
 		(layer "F.Cu")
@@
 	)
 	(segment
-		(start 125.6112 83.4256)
-		(end 125.2419 83.0563)
-		(width 0.25)
-		(layer "F.Cu")
-		(net 4)
-	)
-	(segment
 		(start 139.4361 76.35)
 		(end 139.4361 77.7668)
@@
 	)
 	(segment
-		(start 127.8027 82.9571)
-		(end 129.6723 82.9571)
+		(start 128.426325 82.2)
+		(end 128.4277 82.198625)
 		(width 0.25)
 		(layer "F.Cu")
@@
 	)
 	(segment
-		(start 129.6723 82.1986)
-		(end 129.6723 82.9571)
+		(start 129.7231 83.790208)
+		(end 129.7231 83.9938)
 		(width 0.25)
 		(layer "F.Cu")
@@
 	)
 	(segment
-		(start 126.5881 82.3486)
-		(end 127.1942 82.3486)
+		(start 128.4277 82.494808)
+		(end 129.7231 83.790208)
 		(width 0.25)
 		(layer "F.Cu")
@@
 	)
 	(segment
-		(start 127.1942 82.3486)
-		(end 127.8027 82.9571)
+		(start 128.4277 82.1802)
+		(end 128.4277 82.494808)
 		(width 0.25)
 		(layer "F.Cu")
@@
 	)
 	(segment
-		(start 128.4277 82.1986)
-		(end 128.4277 75.1705)
+		(start 129.6484 74.011778)
+		(end 129.6484 82.174725)
 		(width 0.25)
 		(layer "F.Cu")
@@
 	)
 	(segment
-		(start 128.4277 75.1705)
-		(end 133.0982 70.5)
+		(start 133.160178 70.5)
+		(end 129.6484 74.011778)
 		(width 0.25)
 		(layer "F.Cu")
@@
 	)
 	(segment
-		(start 133.0982 70.5)
-		(end 133.65 70.5)
+		(start 133.65 70.5)
+		(end 133.160178 70.5)
 		(width 0.25)
 		(layer "F.Cu")
@@
 	)
 	(segment
-		(start 148.084 73.8464)
-		(end 148.084 79.2929)
+		(start 129.6484 82.174725)
+		(end 129.6723 82.198625)
 		(width 0.25)
 		(layer "F.Cu")
-		(net 19)
+		(net 18)
 	)
 	(segment
-		(start 148.084 79.2929)
-		(end 147.5554 79.8215)
+		(start 148.084 73.8464)
+		(end 148.084 79.2929)
 		(width 0.25)
 		(layer "F.Cu")
@@
 	)
 	(segment
-		(start 144.25 70.5)
-		(end 144.7376 70.5)
+		(start 148.9723 80.1812)
+		(end 148.9723 82.1802)
 		(width 0.25)
 		(layer "F.Cu")
@@
 	)
 	(segment
-		(start 147.5554 79.8215)
-		(end 147.5554 82.1986)
+		(start 144.25 70.5)
+		(end 144.7376 70.5)
 		(width 0.25)
 		(layer "F.Cu")
@@
 	)
 	(segment
-		(start 149.4667 81.5319)
-		(end 148.8 82.1986)
-		(width 0.25)
-		(layer "F.Cu")
-		(net 20)
-	)
-	(segment
-		(start 151.2933 82.3486)
-		(end 151.2933 81.6865)
-		(width 0.25)
-		(layer "F.Cu")
-		(net 20)
-	)
-	(segment
-		(start 151.1387 81.5319)
-		(end 149.4667 81.5319)
+		(start 148.084 79.2929)
+		(end 148.9723 80.1812)
 		(width 0.25)
 		(layer "F.Cu")
-		(net 20)
+		(net 19)
 	)
 	(segment
-		(start 151.2933 81.6865)
-		(end 151.1387 81.5319)
+		(start 147.7277 82.1802)
+		(end 147.7277 82.8127)
 		(width 0.25)
 		(layer "F.Cu")
@@
 	)
 	(segment
-		(start 152.05 82.3486)
-		(end 151.2933 82.3486)
+		(start 147.7277 82.8127)
+		(end 149.115 84.2)
 		(width 0.25)
 		(layer "F.Cu")
@@
 	)
 	(group ""
-		(members "934e6b23-a1b2-49cb-96a4-2ef338749112" "b1f2cc7d-3c2b-4830-aff2-9c5b7b3e3ec2")
-	)
-	(group ""

Commit message: Order arm encoder board, update bom
Parts:
- D1: footprint LedBlue:YLED0603B -> LedBlue:150080BS75000_Modified
- D2: footprint LedRed:YLED0603R -> LedRed:NCD0603R1
- moved D1 0.15 mm to (128.9, 82.2)
Routing:
- net /BLUE_CATHODE: track 13.7 -> 14.4 mm
Changed lines of the file:
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@@
 		)
 	)
-	(footprint "LedBlue:YLED0603B"
+	(footprint "LedBlue:150080BS75000_Modified"
 		(layer "F.Cu")
-		(at 129.05 82.181575)
+		(at 128.9 82.181575)
+		(tags "150080BS75000 ")
 		(property "Reference" "D1"
-			(at -2.1 0.018425 0)
+			(at 0 0 0)
 			(unlocked yes)
 			(layer "F.SilkS")
+			(hide yes)
 			(effects
 				(font
-					(size 0.7 0.7)
+					(size 1 1)
 					(thickness 0.15)
-					(bold yes)
 				)
 			)
 		)
 		(property "Value" "LEDBLUE"
-			(at -0.01 2.79 0)
+			(at 0 0 0)
 			(unlocked yes)
 			(layer "F.Fab")
@@
 			(effects
 				(font
-					(size 0.7 0.7)
+					(size 1 1)
 					(thickness 0.15)
 				)
@@
 		(property "Datasheet" "~"
 			(at 0 0 0)
-			(unlocked yes)
 			(layer "F.Fab")
 			(hide yes)
 			(effects
 				(font
-					(size 1 1)
+					(size 1.27 1.27)
 					(thickness 0.15)
 				)
@@
 		(property "Description" "Light emitting diode"
 			(at 0 0 0)
-			(unlocked yes)
 			(layer "F.Fab")
 			(hide yes)
 			(effects
 				(font
-					(size 1 1)
+					(size 1.27 1.27)
 					(thickness 0.15)
 				)
@@
 			)
 		)
-		(property "LCSC" "C19171394"
+		(property "LCSC" "C6067133"
 			(at 0 0 0)
-			(layer "F.SilkS")
+			(unlocked yes)
+			(layer "F.Fab")
 			(hide yes)
 			(effects
 				(font
-					(size 1.27 1.27)
+					(size 1 1)
 					(thickness 0.15)
 				)
@@
 		(attr smd)
 		(fp_line
-			(start -0.35 -1.721375)
-			(end 0.24 -1.321375)
-			(stroke
-				(width 0.1)
-				(type default)
-			)
-			(layer "F.SilkS")
-		)
-		(fp_line
-			(start -0.35 -0.921375)
-			(end -0.35 -1.721375)
-			(stroke
-				(width 0.1)
-				(type default)
-			)
-			(layer "F.SilkS")
-		)
-		(fp_line
-			(start 0.24 -1.321375)
-			(end -0.35 -0.921375)
-			(stroke
-				(width 0.1)
-				(type default)
-			)
-			(layer "F.SilkS")
-		)
-		(fp_line
-			(start 0.35 -1.721375)
-			(end 0.35 -0.921375)
-			(stroke
-				(width 0.1)
-				(type default)
-			)
-			(layer "F.SilkS")
-		)
-		(fp_line
-			(start -1.1049 -0.534775)
-			(end 1.1049 -0.534775)
+			(start -0.5 0.8001)
+			(end 0.5 0.8001)
 			(stroke
 				(width 0.1524)
 				(type solid)
 			)
-			(layer "F.CrtYd")
+			(layer "F.SilkS")
 		)
 		(fp_line
-			(start -1.1049 0.532025)
-			(end -1.1049 -0.534775)
+			(start 0.5 -0.8001)
+			(end -0.5 -0.8001)
 			(stroke
 				(width 0.1524)
 				(type solid)
 			)
-			(layer "F.CrtYd")
+			(layer "F.SilkS")
 		)
-		(fp_line
-			(start 1.1049 -0.534775)
-			(end 1.1049 0.532025)
+		(fp_poly
+			(pts
+				(xy -0.3 0) (xy 0.2 -0.4) (xy 0.2 0.4)
+			)
 			(stroke
-				(width 0.1524)
+				(width 0.1)
 				(type solid)
 			)
-			(layer "F.CrtYd")
+			(fill yes)
+			(layer "F.SilkS")
 		)
-		(fp_line
-			(start 1.1049 0.532025)
-			(end -1.1049 0.532025)
+		(fp_rect
+			(start -2 -1)
+			(end 2 1)
 			(stroke
 				(width 0.1524)
 				(type solid)
 			)
+			(fill no)
 			(layer "F.CrtYd")
 		)
 		(fp_line
-			(start -0.8509 -0.458575)
-			(end -0.8509 0.455825)
-			(stroke
-				(width 0.0254)
-				(type solid)
-			)
-			(layer "F.Fab")
-		)
-		(fp_line
-			(start -0.8509 -0.458575)
-			(end -0.8509 0.455825)
-			(stroke
-				(width 0.0254)
-				(type solid)
-			)
-			(layer "F.Fab")
-		)
-		(fp_line
-			(start -0.8509 0.455825)
-			(end -0.2413 0.455825)
-			(stroke
-				(width 0.0254)
-				(type solid)
-			)
-			(layer "F.Fab")
-		)
-		(fp_line
-			(start -0.8509 0.455825)
-			(end 0.8509 0.455825)
+			(start -1.0541 -0.6731)
+			(end -1.0541 0.6731)
 			(stroke
 				(width 0.0254)
@@
 		)
 		(fp_line
-			(start -0.2413 -0.458575)
-			(end -0.8509 -0.458575)
+			(start -1.0541 0.6731)
+			(end 1.0541 0.6731)
 			(stroke
 				(width 0.0254)
@@
 		)
 		(fp_line
-			(start -0.2413 0.455825)
-			(end -0.2413 -0.458575)
+			(start 1.0541 -0.6731)
+			(end -1.0541 -0.6731)
 			(stroke
 				(width 0.0254)
@@
 		)
 		(fp_line
-			(start 0.2413 -0.458575)
-			(end 0.2413 0.455825)
-			(stroke
-				(width 0.0254)
-				(type solid)
-			)
-			(layer "F.Fab")
-		)
-		(fp_line
-			(start 0.2413 0.455825)
-			(end 0.8509 0.455825)
-			(stroke
-				(width 0.0254)
-				(type solid)
-			)
-			(layer "F.Fab")
-		)
-		(fp_line
-			(start 0.8509 -0.458575)
-			(end -0.8509 -0.458575)
-			(stroke
-				(width 0.0254)
-				(type solid)
-			)
-			(layer "F.Fab")
-		)
-		(fp_line
-			(start 0.8509 -0.458575)
-			(end 0.2413 -0.458575)
-			(stroke
-				(width 0.0254)
-				(type solid)
-			)
-			(layer "F.Fab")
-		)
-		(fp_line
-			(start 0.8509 0.455825)
-			(end 0.8509 -0.458575)
-			(stroke
-				(width 0.0254)
-				(type solid)
-			)
-			(layer "F.Fab")
-		)
-		(fp_line
-			(start 0.8509 0.455825)
-			(end 0.8509 -0.458575)
+			(start 1.0541 0.6731)
+			(end 1.0541 -0.6731)
 			(stroke
 				(width 0.0254)
@@
 		)
 		(fp_text user "${REFERENCE}"
-			(at 0 1.348625 0)
+			(at 0 0 0)
 			(unlocked yes)
 			(layer "F.Fab")
 			(effects
 				(font
-					(size 0.7 0.7)
+					(size 1 1)
 					(thickness 0.15)
 				)
@@
 		)
 		(pad "1" smd rect
-			(at 0.6223 -0.001375)
-			(size 0.762 0.8636)
+			(at -1.05 0)
+			(size 1.1 1.3)
 			(layers "F.Cu" "F.Mask" "F.Paste")
 			(net 18 "/BLUE_CATHODE")
@@
 		)
 		(pad "2" smd rect
-			(at -0.6223 -0.001375)
-			(size 0.762 0.8636)
+			(at 1.05 0)
+			(size 1.1 1.3)
 			(layers "F.Cu" "F.Mask" "F.Paste")
 			(net 17 "/BLUE_ANODE")
@@
 			(polygon
 				(pts
-					(xy 128.8595 81.7738) (xy 129.2405 81.7738) (xy 129.2405 82.5866) (xy 128.8595 82.5866)
+					(xy 128.3031 81.559275) (xy 129.4969 81.559275) (xy 129.4969 82.803875) (xy 128.3031 82.803875)
 				)
 			)
 		)
-		(group ""
-			(members "2fce0801-b599-416b-9a28-ec66d2f29070" "4c2caeea-5ffc-4bf9-a038-e9676119c98e"
-				"cb6d4ac6-8f4b-4a35-be16-be7872730078" "e2259e4a-c0e1-4dee-9810-fc8781127cd8"
-			)
-		)
 		(embedded_fonts no)
-		(model "${KIPRJMOD}/dependencies/LedBlue/YLED0603B.stp"
+		(model "${KIPRJMOD}/dependencies/LedBlue/150080BS75000.stp"
 			(offset
 				(xyz 0 0 0)
@@
 		(embedded_fonts no)
 	)
-	(footprint "LedRed:YLED0603R"
+	(footprint "LedRed:NCD0603R1"
 		(layer "F.Cu")
 		(at 148.35 82.1802)
 		(property "Reference" "D2"
-			(at 2.35 0.0198 0)
+			(at 0 -2.52 0)
 			(unlocked yes)
 			(layer "F.SilkS")
@@
 				(font
 					(size 0.7 0.7)
-					(thickness 0.15)
-					(bold yes)
+					(thickness 0.1)
 				)
 			)
@@
 			(unlocked yes)
 			(layer "F.Fab")
-			(hide yes)
 			(effects
 				(font
@@
 			)
 		)
-		(property "LCSC" "C19171390"
+		(property "LCSC" "C84263"
 			(at 0 0 0)
-			(layer "F.SilkS")
+			(unlocked yes)
+			(layer "F.Fab")
 			(hide yes)
 			(effects
 				(font
-					(size 1.27 1.27)
+					(size 1 1)
 					(thickness 0.15)
 				)
@@
 		(attr smd)
 		(fp_line
-			(start -0.35 -1.72)
-			(end 0.24 -1.32)
+			(start -0.305 0.92)
+			(end 0.285 1.32)
 			(stroke
 				(width 0.1)
@@
 		)
 		(fp_line
-			(start -0.35 -0.92)
-			(end -0.35 -1.72)
+			(start -0.305 1.72)
+			(end -0.305 0.92)
 			(stroke
 				(width 0.1)
@@
 		)
 		(fp_line
-			(start 0.24 -1.32)
-			(end -0.35 -0.92)
+			(start 0.285 1.32)
+			(end -0.305 1.72)
 			(stroke
 				(width 0.1)
@@
 		)
 		(fp_line
-			(start 0.35 -1.72)
-			(end 0.35 -0.92)
+			(start 0.395 0.92)
+			(end 0.395 1.72)
 			(stroke
 				(width 0.1)
@@
 		)
 		(group ""
-			(members "2838feab-9907-4163-b272-768ffd1597eb" "37a75fa1-47a7-4eb8-887b-f1942aa10586"
-				"631b936f-8bc4-49c3-b1d9-cb89c1ea0fef" "9073877d-4c01-4eb4-b25a-0fa23aeda077"
+			(members "30b97edd-c802-48e4-ad7d-2dba1fff581d" "89d9f86a-c42d-4938-b2f6-437af3408a9c"
+				"9d839f0e-ddfe-4888-95a7-683de5b0b6ae" "fffa086d-bf4c-4ff8-b41e-7910bfe36def"
 			)
 		)
 		(embedded_fonts no)
-		(model "${KIPRJMOD}/dependencies/LedRed/YLED0603R.stp"
+		(model "${KIPRJMOD}/dependencies/LedRed/NCD0603R1.stp"
 			(offset
 				(xyz 0 0 0)
@@
 		(sheetname "/")
 		(sheetfile "ArmEncoderBoard.kicad_sch")
-		(attr through_hole exclude_from_pos_files)
+		(attr through_hole exclude_from_pos_files exclude_from_bom)
 		(fp_line
 			(start -2.85 -2.75)
@@
 	)
 	(segment
-		(start 128.426325 82.2)
-		(end 128.4277 82.198625)
-		(width 0.25)
-		(layer "F.Cu")
-		(net 17)
-	)
-	(segment
 		(start 129.7231 83.790208)
 		(end 129.7231 83.9938)
@@
 	)
 	(segment
-		(start 128.4277 82.494808)
-		(end 129.7231 83.790208)
+		(start 129.95 83.7669)
+		(end 129.7231 83.9938)
 		(width 0.25)
 		(layer "F.Cu")
@@
 	)
 	(segment
-		(start 128.4277 82.1802)
-		(end 128.4277 82.494808)
+		(start 129.95 82.181575)
+		(end 129.95 83.7669)
 		(width 0.25)
 		(layer "F.Cu")
@@
 	)
 	(segment
-		(start 129.6484 74.011778)
-		(end 129.6484 82.174725)
+		(start 129.6484 82.174725)
+		(end 129.6723 82.198625)
 		(width 0.25)
 		(layer "F.Cu")
-		(net 18)
+		(net 17)
 	)
 	(segment
 		(start 133.160178 70.5)
-		(end 129.6484 74.011778)
+		(end 127.85 75.810178)
 		(width 0.25)
 		(layer "F.Cu")
@@
 	)
 	(segment
-		(start 129.6484 82.174725)
-		(end 129.6723 82.198625)
+		(start 127.85 75.810178)
+		(end 127.85 82.181575)
 		(width 0.25)
 		(layer "F.Cu")

Commit message: Update main and leg board
Parts:
- added C5: 10nF, Capacitor10nF:GRM1885C1H103JA01D, F.Cu at (131.3, 79.5)
- added CR3: BAT54, EnvelopeDiode:BAT54WS-7-F, F.Cu at (126.5, 77.9)
- added D3: LEDRED, LedRed:NCD0603R1, F.Cu at (128.2, 88.6)
- added D4: LEDRED, LedRed:NCD0603R1, F.Cu at (148.5, 88.6)
- added R10: 10K, Resistor10K:CRCW060310K0FKEA, F.Cu at (130.9, 87.5)
- added R11: 10K, Resistor10K:CRCW060310K0FKEA, F.Cu at (145.8, 87.5)
- added R12: 1K, Resistor1K:RCG06031K00FKEA, F.Cu at (145.8, 89.7)
- added R13: 1K, Resistor1K:RCG06031K00FKEA, F.Cu at (130.9, 89.7)
- added R9: 100K, Resistor100K:CRCW0603100KFKEA, F.Cu at (128.6, 77.9)
- moved CR1 2.71 mm to (130.9, 77.2), turned to 180 degrees
- moved J1 0.31 mm to (133.7, 93.5)
- turned D2 to 180 degrees
Connections:
- net Net-(Q1-B) renamed /A_BASE
- net Net-(Q2-B) renamed /I_BASE
- CR1 pad 2: A_BUF -> /A_PULSE
- U2 pad 1: unconnected-(U2-~{MagINC}-Pad1) -> MAGINC
- U2 pad 2: unconnected-(U2-~{MagDEC}-Pad2) -> MAGDEC
Routing:
- net MAGDEC: track 0.00 -> 19.1 mm, vias 0 -> 2
- net MAGINC: track 0.00 -> 13.5 mm, vias 0 -> 2
- net VIN: track 42.6 -> 54.3 mm
- net /A_PULSE: track 0.00 -> 6.17 mm
- net GND: track 23.7 -> 19.8 mm
- net Net-(D3-K): track 0.00 -> 3.15 mm
- net A_BUF: track 8.13 -> 10.2 mm
- net Net-(D4-K): track 0.00 -> 1.83 mm
- net SCK: track 17.1 -> 16.1 mm
- net /A_ENV: track 11.4 -> 12.1 mm
- net /RED_ANODE: track 2.59 -> 2.08 mm
- net /BLUE_CATHODE: track 14.4 -> 14.1 mm, vias 0 -> 2
- net (no net): vias 0 -> 1
Other:
- outline, holes or cut-outs redrawn
- board text added: "MAG+"
- board text added: "MAG-"
