File: boards/ArmRobotBoardTeensy/ArmRobotBoardTeensy.kicad_pcb (KiCad board)
At the start: 2 copper layers, 87.5 x 55 mm, 50 parts, among them J1 B5B-XH-A, J10 B4B-XH-A, J11 B3B-XH-A, J2 B4B-XH-A, J3 B3B-XH-A, J4 B3B-XH-A, J5 B4B-XH-A, J6 B2B-XH-A, J7 B2B-XH-A, J8 B4B-XH-A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

Commit message: Clean up and document boards
Parts:
- added R18: 5.1K, RC0603FR-075K1L:RC0603FR-075K1L, F.Cu at (123.4, 114.6)
- added R19: 5.1K, RC0603FR-075K1L:RC0603FR-075K1L, F.Cu at (147.5, 112.8)
- added R20: 5.1K, RC0603FR-075K1L:RC0603FR-075K1L, F.Cu at (175.2, 118.0)
- D10, D11, D5, D8: value PINK LED -> RED LED; footprint XL-2012UPC:LED_XL-2012SURC_XLG -> NCD0603R1:NCD0603R1
- R10, R12, R13, R5: value 470R -> 1K; footprint RC0603FR-07470RL:RC0603FR-07470RL -> RCG06031K00FKEA:RCG06031K00FKEA
- moved R9 0.54 mm to (123.4, 116.9)
- moved D8 0.25 mm to (110.8, 91.6), turned to 180 degrees
- moved R10 0.25 mm to (115.5, 91.6)
- turned D10 to 180 degrees
- turned D11 to 180 degrees
- turned D5 to 180 degrees
Routing:
- net PWM2VT: track 43.6 -> 70.7 mm
- net PWM1VT: track 34.9 -> 55.1 mm
- net PWM3VT: track 15.5 -> 34.3 mm, vias 0 -> 2
- net GND: track 57.4 -> 45.2 mm, vias 33 -> 35
- net PWM1EN: track 96.5 -> 107.4 mm
- net LPWM1: track 61.3 -> 60.7 mm
- added copper zone on F.Cu, net GND
Other:
- board text added: "3V3"
- board text added: "A"
- board text added: "A0"
- board text added: "A1"
- board text added: "B"
- board text added: "CS"
- board text added: "EN"
- board text added: "GND"
- board text added: "IS"
- board text added: "LIM1"
- board text added: "LIM2"
- board text added: "LPW"
- board text added: "MIS"
- board text added: "RPW"
- board text added: "SCK"
- board text added: "SCL"
- board text added: "SDA"
- board text added: "SIG"
