File: boards/MainRobotBoardTeensy/MainRobotBoardTeensy.kicad_pcb (KiCad board)
At the start: 2 copper layers, 174 x 121.1 mm, 180 parts, among them J1 Screw_Terminal_01x02, J10 B4B-XH-A, J11 IDC, J13 B5B-XH-A, J14 B5B-XH-A, J2 B3B-XH-A, J3 B3B-XH-A, J4 B3B-XH-A, J5 B3B-XH-A, J6 B3B-XH-A, J7 B3B-XH-A, J8 B3B-XH-A, J9 B3B-XH-A, Q1 AO3400A, Q10 AO3400A, Q11 AO3400A, Q12 AO3400A, Q13 AO3400A, Q14 AO3400A, Q15 AO3400A, Q16 AO3400A, Q17 AO3400A, Q18 AO3400A, Q19 AO3400A, Q2 AO3400A, Q20 AO3400A, Q3 AO3400A, Q4 AO3400A, Q5 AO3400A, Q6 AO3400A, Q7 AO3400A, Q8 AO3400A, Q9 AO3400A, U1 Teensy4.0, U10 KWL-R1025BB, U11 SSD1306, U2 TLC555CDR, U3 SN74HC08DR, U4 SN74HC08DR, U6 SN74HC08DR, U7 ACS37220, U8 SN74HC595DR, U9 SN74HC595DR

Commit message: Re-designing main board
Parts:
- removed C7, C8: 100nF, Capacitor100nF:CC0603KRX7R9BB104
- removed D7, D8: REDLED, LedRed:NCD0603R1
- removed J13, J14: B5B-XH-A, Connector_JST:JST_XH_B5B-XH-A_1x05_P2.50mm_Vertical
- removed J4: B3B-XH-A, Connector_JST:JST_XH_B3B-XH-A_1x03_P2.50mm_Vertical
- removed Q7, Q8: AO3400A, AO3400A:AO3400A
- removed R10: 1K, Resistor1K:RCG06031K00FKEA
- removed R54, R55, R70, R72: 10K, Resistor10K:CRCW060310K0FKEA
- removed R56, R57: 47R, Resistor47:RESC1608X55
- removed R71, R73: 100K, Resistor100K:CRCW0603100KFKEA
- removed U9: SN74HC595DR, ShiftRegister:SN74HC595DR
- added U5: PCA9685PW_118, PWMDriver:PCA9685PW,118, F.Cu at (157.7, 100.7)
- R3, R4, R5, R6, R7, R8: value 1K -> 470R
- R9: value 1K -> 10K; footprint Resistor1K:RCG06031K00FKEA -> Resistor10K:CRCW060310K0FKEA
- U1: value Teensy4.0 -> Teensy4.1; footprint Teensy:Teensy40 -> Teensy4.1:Teensy41
- U8: value SN74HC595DR -> SSD1306; footprint ShiftRegister:SN74HC595DR -> SSD1306:SSD1306
- moved D17 136.2 mm to (77.5, 117.3)
- moved D18 136.2 mm to (84.3, 117.3)
- moved D5 136.2 mm to (80.9, 117.3)
- moved J11 136.2 mm to (77.0, 111.6)
- moved R100 110.5 mm to (205.5, 150.8)
- moved R101 110.5 mm to (205.5, 148.3)
- moved R102 110.5 mm to (205.5, 145.7)
- moved R103 110.5 mm to (205.5, 143.2)
- moved R104 110.5 mm to (205.5, 140.6)
- moved R105 110.5 mm to (205.5, 138.1)
- moved R106 110.5 mm to (205.5, 135.5)
- moved R107 110.5 mm to (205.5, 132.9)
- moved R98 110.5 mm to (205.5, 155.9)
- moved R99 110.5 mm to (205.5, 153.4)
- moved U10 110.5 mm to (212.3, 144.4)
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Connections:
- net TORSO1 renamed TORSO
- C1 pad 2: GND -> V-
- C10 pad 1: GND -> V-
- C2 pad 2: GND -> V-
- C3 pad 2: GND -> V-
- C4 pad 2: GND -> V-
- C5 pad 2: GND -> V-
- J11 pad 2: GND -> V-
- J11 pad 4: GND -> V-
- J11 pad 6: GND -> V-
- J11 pad 8: GND -> V-
- J2 pad 3: GND -> V-
- J3 pad 3: GND -> V-
- J9 pad 3: GND -> V-
- Q1 pad 2: GND -> V-
- Q10 pad 2: GND -> V-
- Q11 pad 2: GND -> V-
- Q12 pad 2: GND -> V-
- Q13 pad 2: GND -> V-
- Q14 pad 2: GND -> V-
- Q15 pad 2: GND -> V-
- Q16 pad 2: GND -> V-
- Q17 pad 2: GND -> V-
- Q18 pad 2: GND -> V-
- Q19 pad 2: GND -> V-
- Q2 pad 2: GND -> V-
- Q20 pad 2: GND -> V-
- Q3 pad 2: GND -> V-
- Q4 pad 2: GND -> V-
- Q5 pad 2: GND -> V-
- Q6 pad 2: GND -> V-
- Q9 pad 2: GND -> V-
- R38 pad 2: GND -> V-
- R39 pad 2: GND -> V-
- R40 pad 2: GND -> V-
- R41 pad 2: GND -> V-
- R42 pad 2: GND -> V-
- R43 pad 2: GND -> V-
- R44 pad 2: GND -> V-
- R45 pad 2: GND -> V-
- R46 pad 2: GND -> V-
- R47 pad 2: GND -> V-
- R48 pad 2: GND -> V-
- R49 pad 1: TORSOPANEN -> V-
- R49 pad 2: GND -> TORSOPANEN
- R50 pad 2: GND -> V-
- R51 pad 2: GND -> V-
- R52 pad 2: GND -> V-
- R53 pad 2: GND -> V-
- R75 pad 2: GND -> V-
- R77 pad 2: GND -> V-
- R79 pad 2: GND -> V-
- R81 pad 2: GND -> V-
- R83 pad 2: GND -> V-
- R85 pad 2: GND -> V-
- R87 pad 2: GND -> V-
- R89 pad 2: GND -> V-
- R9 pad 2: +3.3V -> V-
- R91 pad 2: GND -> V-
- R93 pad 2: GND -> V-
- R95 pad 2: GND -> V-
- R97 pad 2: GND -> V-
- U1 pad 1: GND -> V-
- U1 pad 10: TORSOPANST -> TORSOTILT2EN
- U1 pad 11: TORSOTILT1LPWM -> LED1
- U1 pad 12: TORSOTILT1RPWM -> LED2
- U1 pad 13: MOSI -> unconnected-(U1-11_MOSI_CTX1-Pad13)
- U1 pad 14: Net-(U1-12_MISO_MQSL) -> unconnected-(U1-12_MISO_MQSL-Pad14)
- U1 pad 15: unconnected-(U1-VBAT-Pad15) -> +3.3V
- U1 pad 16: +3.3V -> LED7
- U1 pad 17: GND -> LED8
- U1 pad 18: unconnected-(U1-PROGRAM-Pad18) -> LED9
- U1 pad 19: unconnected-(U1-ON_OFF-Pad19) -> LED10
- U1 pad 2: CSHEAD -> HEADPANEN
- U1 pad 20: Net-(U1-13_SCK_CRX1_LED) -> unconnected-(U1-28_RX7-Pad20)
- U1 pad 21: CURRENT -> unconnected-(U1-29_TX7-Pad21)
- U1 pad 22: HEAD -> unconnected-(U1-30_CRX3-Pad22)
- U1 pad 23: Net-(U1-16_A2_RX4_SCL1) -> unconnected-(U1-31_CTX3-Pad23)
- U1 pad 24: VSENSE -> unconnected-(U1-32_OUT1B-Pad24)
- U1 pad 25: SDA -> unconnected-(U1-33_MCLK2-Pad25)
- U1 pad 26: SCL -> unconnected-(U1-34_RX8-Pad26)
- U1 pad 27: TORSOPANDIR -> unconnected-(U1-35_TX8-Pad27)
- U1 pad 28: TORSOPANPWM -> unconnected-(U1-36_CS-Pad28)
- U1 pad 29: TORSOTILT2LPWM -> unconnected-(U1-37_CS-Pad29)
- U1 pad 3: CSTORSO -> HEADPANDIR
- U1 pad 30: TORSOTILT2RPWM -> unconnected-(U1-38_CS1_IN1-Pad30)
- U1 pad 34: unconnected-(U1-VUSB-Pad34) -> V-
- U1 pad 35: HEADPANPUL -> unconnected-(U1-13_SCK_LED-Pad35)
- U1 pad 36: HEADPANDIR -> CURRENT
- U1 pad 37: MOUTHSERVO -> HEAD
- U1 pad 38: HEADTILT1EN -> Net-(U1-16_A2_RX4_SCL1)
- U1 pad 39: HEADTILT2EN -> VSENSE
- U1 pad 4: HEADTILT1LPWM -> TORSOPANEN
- U1 pad 40: TORSOTILT1EN -> SDA
- U1 pad 41: TORSOTILT2EN -> SCL
- U1 pad 42: RCLK -> LED3
- U1 pad 43: unconnected-(U1-32_OUT1B-Pad43) -> LED4
- U1 pad 44: unconnected-(U1-33_MCLK2-Pad44) -> LED5
- U1 pad 5: HEADTILT1RPWM -> TORSOPANDIR
- U1 pad 6: HEADTILT2LPWM -> TORSOPANST
- U1 pad 7: HEADTILT2RPWM -> HEADTILT1EN
- U1 pad 8: HEADPANEN -> HEADTILT2EN
- U1 pad 9: TORSOPANEN -> TORSOTILT1EN
- U11 pad 2: GND -> V-
- U2 pad 1: GND -> V-
- U3 pad 7: GND -> V-
- U4 pad 7: GND -> V-
- U6 pad 7: GND -> V-
- U7 pad 2: GND -> V-
- U8 pad 1: LED2 -> +3.3V
- U8 pad 2: LED3 -> V-
- U8 pad 3: LED4 -> SCL
- U8 pad 4: LED5 -> SDA
Routing:
- net +3.3V: track 643.9 -> 0.00 mm
- net TORSO: track 181.8 -> 0.00 mm, vias 2 -> 0
- net TORSOENCODERST: track 176.8 -> 0.00 mm, vias 4 -> 0
- net Net-(J5-Pin_3): track 173.7 -> 0.00 mm, vias 5 -> 0
- net HEADENCODERST: track 169.5 -> 0.00 mm, vias 2 -> 0
- net SCK: track 169.4 -> 0.00 mm, vias 5 -> 0
- net Net-(J5-Pin_2): track 168.5 -> 0.00 mm, vias 4 -> 0
- net Net-(D8-A): track 163.2 -> 0.00 mm
- net Net-(J7-Pin_2): track 149.8 -> 0.00 mm, vias 3 -> 0
- net HEADTILT1EN: track 146.4 -> 0.00 mm, vias 5 -> 0
- net CSHEAD: track 145.9 -> 0.00 mm, vias 1 -> 0
- net Net-(J6-Pin_3): track 145.8 -> 0.00 mm, vias 5 -> 0
- net HEADTILT1RPWM: track 141.5 -> 0.00 mm, vias 5 -> 0
- net HEADTILT1LPWM: track 134.1 -> 0.00 mm, vias 3 -> 0
- net Net-(J6-Pin_2): track 131.0 -> 0.00 mm, vias 4 -> 0
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- added copper zone on B.Cu, net V-
- added copper zone on F.Cu, net V-
- removed copper zone on B.Cu, net GND
- removed copper zone on F.Cu, net GND
Other:
- board text added: "01binary"
- board text added: "BATTERY"
- board text added: "CURRENT SENSE"
- board text added: "POWER"
- board text added: "TORSO TILT"
- board text added: "VOLTAGE SENSE"
- board text added: "VOLTAGE/CURRENT"
- board text added: "motors"
- board text added: "servo / stepper"
- board text added: "tech art"
- board text removed: "ANALOG"
- board text removed: "CS"
- board text removed: "D0"
- board text removed: "D1"
- board text removed: "DIGITAL"
- board text removed: "MIS"
- board text removed: "MOTORS"
- board text removed: "OLED DISPLAY"
- board text removed: "SCK"
- board text removed: "SERVOS AND STEPPERS"
- board text removed: "SSD1306"
- board text removed: "actuators"

Commit message: Pre-flight main board
Parts:
- removed R9: 10K, Resistor10K:CRCW060310K0FKEA
- added U9: 74HCT125D, LevelShifter:74HCT125D, F.Cu at (113.7, 101.4)
- D1, D2, D3, D4, D5, D6: footprint LedRed:NCD0603R1 -> LedRed:XL-1608SURC-06
- R3, R4, R5, R6, R7, R8: footprint Resistor1K:RCG06031K00FKEA -> Resistor470:RC0603FR-07470RL
- U5: value PCA9685PW_118 -> 74HCT125D; footprint PWMDriver:PCA9685PW,118 -> LevelShifter:74HCT125D
- moved U5 31.7 mm to (126.0, 101.2), turned to 0 degrees
- moved C1 8.53 mm to (140.3, 104.5)
- moved C2 8.53 mm to (151.0, 104.8)
- moved R1 8.53 mm to (140.2, 101.8)
- moved R2 8.53 mm to (151.6, 101.8)
- moved U2 8.53 mm to (145.9, 102.5)
- moved U3 4.46 mm to (135.5, 114.9)
- moved U6 4.46 mm to (145.9, 114.9)
- moved U4 4.46 mm to (156.3, 114.9)
- moved R7 3.25 mm to (100.4, 108.9)
- moved R22 3.23 mm to (126.1, 108.9)
- moved R96 3.23 mm to (126.1, 116.4)
- moved R21 3.23 mm to (113.8, 108.9)
- moved R68 3.23 mm to (120.0, 116.4)
- moved R94 3.23 mm to (113.8, 116.4)
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Connections:
- J10 pad 3: HEADPANDIR -> HEADPANDIR5V
- J10 pad 4: HEADPANEN -> HEADPANEN5V
- J11 pad 1: TORSOPANEN -> TORSOPANEN5V
- J11 pad 3: TORSOPANDIR -> TORSOPANDIR5V
- J11 pad 7: TORSOPANST -> unconnected-(J11-Pin_7-Pad7)
- R100 pad 2: +3.3V -> LED3
- R101 pad 2: +3.3V -> LED4
- R102 pad 2: +3.3V -> LED5
- R103 pad 2: +3.3V -> LED6
- R104 pad 2: +3.3V -> LED7
- R105 pad 2: +3.3V -> LED8
- R106 pad 2: +3.3V -> LED9
- R107 pad 2: +3.3V -> LED10
- R32 pad 2: TORSOPANPWM -> TORSOPANPWM5V
- R33 pad 2: HEADPANPUL -> HEADPANPUL5V
- R48 pad 1: HEADPANEN -> HEADPANEN5V
- R49 pad 2: TORSOPANEN -> TORSOPANEN5V
- R98 pad 2: +3.3V -> LED1
- R99 pad 2: +3.3V -> LED2
- U1 pad 10: TORSOTILT2EN -> HEADTILT2EN
- U1 pad 11: LED1 -> HEADTILT1LPWM
- U1 pad 12: LED2 -> HEADTILT1RPWM
- U1 pad 13: unconnected-(U1-11_MOSI_CTX1-Pad13) -> HEADTILT2LPWM
- U1 pad 14: unconnected-(U1-12_MISO_MQSL-Pad14) -> HEADTILT2RPWM
- U1 pad 16: LED7 -> LED1
- U1 pad 17: LED8 -> LED2
- U1 pad 18: LED9 -> LED3
- U1 pad 19: LED10 -> LED4
- U1 pad 20: unconnected-(U1-28_RX7-Pad20) -> TORSOTILT2LPWM
- U1 pad 21: unconnected-(U1-29_TX7-Pad21) -> TORSOTILT2RPWM
- U1 pad 22: unconnected-(U1-30_CRX3-Pad22) -> LED5
- U1 pad 23: unconnected-(U1-31_CTX3-Pad23) -> LED6
- U1 pad 24: unconnected-(U1-32_OUT1B-Pad24) -> LED7
- U1 pad 25: unconnected-(U1-33_MCLK2-Pad25) -> LED8
- U1 pad 26: unconnected-(U1-34_RX8-Pad26) -> LED9
- U1 pad 27: unconnected-(U1-35_TX8-Pad27) -> LED10
- U1 pad 28: unconnected-(U1-36_CS-Pad28) -> MOUTHSERVO
- U1 pad 4: TORSOPANEN -> HEADPANPUL
- U1 pad 42: LED3 -> TORSOTILT1EN
- U1 pad 43: LED4 -> TORSOTILT2EN
- U1 pad 44: LED5 -> TORSOTILT1LPWM
- U1 pad 45: LED6 -> TORSOTILT1RPWM
- U1 pad 46: unconnected-(U1-3V3-Pad46) -> +3.3V
- U1 pad 49: unconnected-(U1-VUSB-Pad49) -> +5V
- U1 pad 5: TORSOPANDIR -> TORSOPANEN
- U1 pad 6: TORSOPANST -> TORSOPANDIR
- U1 pad 7: HEADTILT1EN -> TORSOPANPWM
- U1 pad 8: HEADTILT2EN -> unconnected-(U1-6_OUT1D-Pad8)
- U1 pad 9: TORSOTILT1EN -> HEADTILT1EN
- U10 pad 1: LED1 -> V-
- U10 pad 10: LED10 -> V-
- U10 pad 2: LED2 -> V-
- U10 pad 3: LED3 -> V-
- U10 pad 4: LED4 -> V-
- U10 pad 5: LED5 -> V-
- U10 pad 6: LED6 -> V-
- U10 pad 7: LED7 -> V-
- U10 pad 8: LED8 -> V-
- U10 pad 9: LED9 -> V-
- U5 pad 10: HEADTILT2LPWM -> V-
- U5 pad 11: HEADTILT2RPWM -> unconnected-(U5-4Y-Pad11)
- U5 pad 12: TORSOTILT1LPWM -> unconnected-(U5-4A-Pad12)
- U5 pad 13: TORSOTILT1RPWM -> +5V
- U5 pad 14: V- -> +5V
- U5 pad 2: V- -> HEADPANEN
- U5 pad 3: V- -> HEADPANEN5V
- U5 pad 5: V- -> HEADPANPUL
- U5 pad 6: TORSOPANPWM -> HEADPANPUL5V
- U5 pad 7: HEADPANPUL -> V-
- U5 pad 8: HEADTILT1LPWM -> HEADPANDIR5V
- U5 pad 9: HEADTILT1RPWM -> HEADPANDIR
Routing:
- net +3.3V: track 0.00 -> 564.5 mm
- net HEADPANPUL: track 0.00 -> 198.7 mm, vias 0 -> 3
- net TORSOPANEN: track 0.00 -> 182.6 mm, vias 0 -> 3
- net TORSOPANDIR: track 0.00 -> 178.5 mm, vias 0 -> 4
- net HEADPANEN: track 0.00 -> 170.1 mm, vias 0 -> 3
- net HEADTILT1EN: track 0.00 -> 164.0 mm, vias 0 -> 4
- net Net-(J2-Pin_2): track 0.00 -> 150.5 mm, vias 0 -> 4
- net TORSO: track 0.00 -> 150.0 mm, vias 0 -> 3
- net Net-(J11-Pin_5): track 0.00 -> 141.7 mm, vias 0 -> 3
- net Net-(J9-Pin_1): track 0.00 -> 141.1 mm, vias 0 -> 3
- net SDA: track 0.00 -> 139.8 mm, vias 0 -> 3
- net +5V: track 0.00 -> 136.4 mm, vias 0 -> 4
- net SCL: track 0.00 -> 133.7 mm, vias 0 -> 2
- net TORSOPANPWM5V: track 0.00 -> 128.4 mm, vias 0 -> 8
- net HEADPANDIR: track 0.00 -> 125.6 mm, vias 0 -> 3
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Other:
- board text added: "METERS"
- board text removed: "A3"
- board text removed: "CURRENT SENSE"
- board text removed: "D2/D3"
- board text removed: "D20/21"
- board text removed: "D22/23"
- board text removed: "D24/25"
- board text removed: "D26"
- board text removed: "D27"
- board text removed: "D28"
- board text removed: "D29"
- board text removed: "D30"
- board text removed: "D4/D5"
- board text removed: "D6"
- board text removed: "D7"
- board text removed: "D9/10"
- board text removed: "DIR PWM"
- board text removed: "POWER"
- board text removed: "PUL DIR"
- board text removed: "VOLTAGE SENSE"
- board text removed: "VOLTAGE/CURRENT"
