File: boards/MainRobotBoardTeensy/MainRobotBoardTeensy.kicad_pcb (KiCad board)
At the start: 2 copper layers, 174 x 121.1 mm, 162 parts, among them J1 Screw_Terminal_01x02, J10 B4B-XH-A, J11 IDC, J2 B3B-XH-A, J3 B3B-XH-A, J5 B3B-XH-A, J6 B3B-XH-A, J7 B3B-XH-A, J8 B3B-XH-A, J9 B3B-XH-A, Q1 AO3400A, Q10 AO3400A, Q11 AO3400A, Q12 AO3400A, Q13 AO3400A, Q14 AO3400A, Q15 AO3400A, Q16 AO3400A, Q17 AO3400A, Q18 AO3400A, Q19 AO3400A, Q2 AO3400A, Q20 AO3400A, Q3 AO3400A, Q4 AO3400A, Q5 AO3400A, Q6 AO3400A, Q9 AO3400A, U1 Teensy4.1, U10 KWL-R1025BB, U11 SSD1306, U2 TLC555CDR, U3 SN74HC08DR, U4 SN74HC08DR, U5 74HCT125D, U6 SN74HC08DR, U7 ACS37220, U8 SSD1306, U9 74HCT125D

Commit message: Main robot board 5V and 7V routing
Parts:
- added J4: Screw_Terminal_01x02, TerminalBlock_Phoenix:TerminalBlock_Phoenix_MKDS-1,5-2-5.08_1x02_P5.08mm_Horizontal, F.Cu at (221.4, 137.0)
- moved R46 89.8 mm to (75.9, 99.8)
- moved R31 89.5 mm to (79.3, 99.8)
Connections:
- J10 pad 1: +3.3V -> +5V
- J9 pad 2: +3.3V -> +7.5V
- R31 pad 2: MOUTHSERVO -> MOUTHSERVO5V
- U5 pad 11: unconnected-(U5-4Y-Pad11) -> MOUTHSERVO5V
- U5 pad 12: unconnected-(U5-4A-Pad12) -> MOUTHSERVO
- U5 pad 13: +5V -> V-
Routing:
- net +7.5V: track 0.00 -> 202.2 mm
- net MOUTHSERVO: track 14.2 -> 154.4 mm
- net Net-(J9-Pin_1): track 141.1 -> 6.71 mm, vias 3 -> 0
- net +3.3V: track 564.5 -> 486.2 mm, vias 0 -> 1
- net MOUTHSERVO5V: track 0.00 -> 63.8 mm, vias 0 -> 2
- net +5V: track 136.4 -> 148.4 mm
- net V-: track 59.2 -> 62.6 mm, vias 59 -> 79
Other:
- board text added: "24V"
- board text added: "24V 100A"
- board text added: "5V"
- board text added: "7V"
- board text added: "BATTERY CHARGE"
- board text added: "CURRENT SENSE"
- board text added: "POWER"
- board text added: "SERVO 7V"
- board text added: "VOLTAGE / CURRENT"
- board text added: "VOLTAGE SENSE"
- board text added: "developed at CTRL^H hackerspace"
- board text removed: "BATTERY"
