File: boards/MainRobotBoardTeensy/MainRobotBoardTeensy.kicad_sch (KiCad schematic)
At the start: 176 parts, among them J10 B4B-XH-A, J11 IDC, J13 B5B-XH-A, J14 B5B-XH-A, J2 B3B-XH-A, J3 B3B-XH-A, J4 B3B-XH-A, J5 B3B-XH-A, J6 B3B-XH-A, J7 B3B-XH-A, J8 B3B-XH-A, J9 B3B-XH-A, Q1 AO3400A, Q10 AO3400A, Q11 AO3400A, Q12 AO3400A, Q13 AO3400A, Q14 AO3400A, Q15 AO3400A, Q16 AO3400A, Q17 AO3400A, Q18 AO3400A, Q19 AO3400A, Q2 AO3400A, Q20 AO3400A, Q3 AO3400A, Q4 AO3400A, Q5 AO3400A, Q6 AO3400A, Q7 AO3400A, Q8 AO3400A, Q9 AO3400A, U1 Teensy4.0, U10 KWL-R1025BB, U11 SSD1306, U2 TLC555CDR, U3 SN74HC08DR, U4 SN74HC08DR, U5 INA260, U6 SN74HC08DR, U7 ACS37220, U8 SN74HC595DR, U9 SN74HC595DR

Commit message: Final board export after testing
Parts:
- R100, R101, R102, R103, R104, R105, R106, R107, R98, R99: value 150R -> 470R; footprint Resistor150:RESC1607X60N -> Resistor470:RC0603FR-07470RL; LCSC C114608 -> C114669
Changed lines of the file:
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@@
 			)
 		)
-		(property "Value" "150R"
+		(property "Value" "470R"
 			(at 496.57 334.01 90)
 			(effects
@@
 			)
 		)
-		(property "Footprint" "Resistor150:RESC1607X60N"
+		(property "Footprint" "Resistor470:RC0603FR-07470RL"
 			(at 471.424 341.884 90)
 			(effects
@@
 			)
 		)
-		(property "LCSC" "C114608"
+		(property "LCSC" "C114669"
 			(at 471.17 336.55 0)
 			(effects
@@
 				)
 				(justify left)
+				(hide yes)
 			)
 		)
-		(property "Value" "150R"
+		(property "Value" "470R"
 			(at 478.79 360.68 90)
 			(effects
@@
 				)
 				(justify left)
+				(hide yes)
 			)
 		)
-		(property "Footprint" "Resistor150:RESC1607X60N"
+		(property "Footprint" "Resistor470:RC0603FR-07470RL"
 			(at 471.424 357.124 90)
 			(effects
@@
 			)
 		)
-		(property "LCSC" "C114608"
+		(property "LCSC" "C114669"
 			(at 471.17 351.79 0)
 			(effects
@@
 			)
 		)
-		(property "Value" "150R"
+		(property "Value" "470R"
 			(at 496.57 356.87 90)
 			(effects
@@
 			)
 		)
-		(property "Footprint" "Resistor150:RESC1607X60N"
+		(property "Footprint" "Resistor470:RC0603FR-07470RL"
 			(at 471.424 349.504 90)
 			(effects
@@
 			)
 		)
-		(property "LCSC" "C114608"
+		(property "LCSC" "C114669"
 			(at 471.17 344.17 0)
 			(effects
@@
 			)
 		)
-		(property "Value" "150R"
+		(property "Value" "470R"
 			(at 481.33 328.93 90)
 			(effects
@@
 			)
 		)
-		(property "Footprint" "Resistor150:RESC1607X60N"
+		(property "Footprint" "Resistor470:RC0603FR-07470RL"
 			(at 471.424 336.804 90)
 			(effects
@@
 			)
 		)
-		(property "LCSC" "C114608"
+		(property "LCSC" "C114669"
 			(at 471.17 331.47 0)
 			(effects
@@
 		(dnp no)
 		(property "Reference" "R98"
-			(at 477.52 332.74 90)
+			(at 472.44 331.47 90)
 			(effects
 				(font
@@
 			)
 		)
-		(property "Value" "150R"
-			(at 477.52 330.2 90)
+		(property "Value" "470R"
+			(at 472.44 328.93 90)
 			(effects
 				(font
@@
 			)
 		)
-		(property "Footprint" "Resistor150:RESC1607X60N"
+		(property "Footprint" "Resistor470:RC0603FR-07470RL"
 			(at 471.424 334.264 90)
 			(effects
@@
 			)
 		)
-		(property "LCSC" "C114608"
+		(property "LCSC" "C114669"
 			(at 471.17 328.93 0)
 			(effects
@@
 			)
 		)
-		(property "Value" "150R"
+		(property "Value" "470R"
 			(at 481.33 361.95 90)
 			(effects
@@
 			)
 		)
-		(property "Footprint" "Resistor150:RESC1607X60N"
+		(property "Footprint" "Resistor470:RC0603FR-07470RL"
 			(at 471.424 354.584 90)
 			(effects
@@
 			)
 		)
-		(property "LCSC" "C114608"
+		(property "LCSC" "C114669"
 			(at 471.17 349.25 0)
 			(effects
@@
 			)
 		)
-		(property "Value" "150R"
+		(property "Value" "470R"
 			(at 504.19 354.33 90)
 			(effects
@@
 			)
 		)
-		(property "Footprint" "Resistor150:RESC1607X60N"
+		(property "Footprint" "Resistor470:RC0603FR-07470RL"
 			(at 471.424 346.964 90)
 			(effects
@@
 			)
 		)
-		(property "LCSC" "C114608"
+		(property "LCSC" "C114669"
 			(at 471.17 341.63 0)
 			(effects
@@
 			)
 		)
-		(property "Value" "150R"
+		(property "Value" "470R"
 			(at 488.95 331.47 90)
 			(effects
@@
 			)
 		)
-		(property "Footprint" "Resistor150:RESC1607X60N"
+		(property "Footprint" "Resistor470:RC0603FR-07470RL"
 			(at 471.424 339.344 90)
 			(effects
@@
 			)
 		)
-		(property "LCSC" "C114608"
+		(property "LCSC" "C114669"
 			(at 471.17 334.01 0)
 			(effects
@@
 			)
 		)
-		(property "Value" "150R"
+		(property "Value" "470R"
 			(at 504.19 336.55 90)
 			(effects
@@
 			)
 		)
-		(property "Footprint" "Resistor150:RESC1607X60N"
+		(property "Footprint" "Resistor470:RC0603FR-07470RL"
 			(at 471.424 344.424 90)
 			(effects
@@
 			)
 		)
-		(property "LCSC" "C114608"
+		(property "LCSC" "C114669"
 			(at 471.17 339.09 0)
 			(effects
@@
 			)
 		)
-		(property "Value" "150R"
+		(property "Value" "470R"
 			(at 488.95 359.41 90)
 			(effects
@@
 			)
 		)
-		(property "Footprint" "Resistor150:RESC1607X60N"
+		(property "Footprint" "Resistor470:RC0603FR-07470RL"
 			(at 471.424 352.044 90)
 			(effects
@@
 			)
 		)
-		(property "LCSC" "C114608"
+		(property "LCSC" "C114669"
 			(at 471.17 346.71 0)
 			(effects

Commit message: Leg board re-do LED displays, main board prepare for re-routing
Parts:
- removed C6: 47nF, Capacitor47nF:CAPC1608X90N, symbol CC0603JRX7R7BB105:CC0603JRX7R7BB105
- removed R37: 2.2K, Resistor2.2K:RC0603FR-072K2L, symbol Device:R_US
- removed U5: INA260, INA260:INA260, symbol INA260:INA260
- added C10: 10nF, Capacitor0.01uF:C0402C103J4RACTU, symbol C0402C103J4RACTU:C0402C103J4RACTU
- added C9: 100nF, Capacitor100nF:CC0603KRX7R9BB104, symbol CC0603JRX7R7BB105:CC0603JRX7R7BB105
- added J1: Screw_Terminal_01x02, TerminalBlock_Phoenix:TerminalBlock_Phoenix_MKDS-1,5-2-5.08_1x02_P5.08mm_Horizontal, symbol Connector:Screw_Terminal_01x02
- added R59, R61: 100K, Resistor100K:CRCW0603100KFKEA, symbol Device:R_US
- added R63: 22K, Resistor22K:0603WAF2202T5E, symbol Device:R_US
- added R65: 1K, Resistor1K:RCG06031K00FKEA, symbol Device:R_US
Connections:
- net GND: now also C10.1
- net TORSO1: now also C5.1, J3.2 (Pin_2), J4.2 (Pin_2), R36.1; no longer R36.2, U1.23 (16_A2_RX4_SCL1)
- net TORSO2 renamed VSENSE
- net VSENSE: now also C10.2, R65.1
- new net: C9.2, R61.1, R63.1, R65.2
- new net: R59.1, R61.2
- new net: R36.2, U1.23 (16_A2_RX4_SCL1)
- new net V+: J1.1 (Pin_1), R59.2
- new net V-: C9.1, J1.2 (Pin_2), R63.2
Other:
- note added: "Current Sensing"
- note added: "EMPTY"
- note added: "FULL"
- note added: "Voltage Sensing"
- note removed: "Current Sensor"
- note removed: "Voltage Sensor"
- moved on the sheet: C5, R100, R101, R102, R103, R104, R105, R106, R36, R98, R99, U10

Commit message: Re-designing main board
Parts:
- removed C7, C8: 100nF, Capacitor100nF:CC0603KRX7R9BB104, symbol CC0603JRX7R7BB105:CC0603JRX7R7BB105
- removed D7, D8: REDLED, LedRed:NCD0603R1, symbol Device:LED
- removed J13, J14: B5B-XH-A, Connector_JST:JST_XH_B5B-XH-A_1x05_P2.50mm_Vertical, symbol Connector_Generic:Conn_01x05
- removed J4: B3B-XH-A, Connector_JST:JST_XH_B3B-XH-A_1x03_P2.50mm_Vertical, symbol Connector_Generic:Conn_01x03
- removed Q7, Q8: AO3400A, AO3400A:AO3400A, symbol AO3400A:AO3400A
- removed R10: 1K, Resistor1K:RCG06031K00FKEA, symbol Device:R_US
- removed R54, R55, R70, R72: 10K, Resistor10K:CRCW060310K0FKEA, symbol Device:R_US
- removed R56, R57: 47R, Resistor47:RESC1608X55, symbol Device:R_US
- removed R71, R73: 100K, Resistor100K:CRCW0603100KFKEA, symbol Device:R_US
- removed U1: Teensy4.0, Teensy:Teensy40, symbol Teensy:Teensy4.0
- removed U8, U9: SN74HC595DR, ShiftRegister:SN74HC595DR, symbol ShiftRegister:SN74HC595DR
- added U1: Teensy4.1, Teensy4.1:Teensy41, symbol Teensy4.1:Teensy4.1
- added U5: PCA9685PW_118, PWMDriver:PCA9685PW,118, symbol PWMDriver:PCA9685PW_118
- added U8: SSD1306, SSD1306:SSD1306, symbol SSD1306:SSD1306
- D1, D2, D3, D4, D5, D6: footprint LedRed:NCD0603R1 -> LedRed:XL-1608SURC-06; LCSC C84263 -> C965799
- R3, R4, R5, R6, R7, R8: value 1K -> 470R; footprint Resistor1K:RCG06031K00FKEA -> Resistor470:RC0603FR-07470RL; LCSC C4264491 -> C114669
- R9: value 1K -> 10K; footprint Resistor1K:RCG06031K00FKEA -> Resistor10K:CRCW060310K0FKEA; LCSC C4264491 -> C844918
Connections:
- net V- is gone; now on net GND: C9.1, J1.2 (Pin_2), R63.2
- net +3.3V: now also U1.15 (3V3), U1.51 (3V3), U5.28 (VDD), U8.1 (VCC); no longer R9.2
- net CURRENT: now also U1.36 (14_A0_TX3_SPDIF_OUT)
- net GND: now also R49.1, R9.2, U1.1 (GND), U1.34 (GND), U1.47 (GND), U1.52 (GND), U5.1 (A0), U5.14 (VSS), U5.2 (A1), U5.24 (A5), U5.25 (EXTCLK), U5.3 (A2), U5.4 (A3), U5.5 (A4), U8.2 (GND); no longer R49.2
- net HEAD: now also U1.37 (15_A1_RX3_SPDIF_IN)
- net HEADPANDIR: now also U1.3 (1_TX1_CTX2_MISO1)
- net HEADPANEN: now also U1.2 (0_RX1_CRX2_CS1)
- net HEADPANPUL: now also U5.7 (LED1)
- net HEADTILT1EN: now also U1.7 (5_IN2)
- net HEADTILT1LPWM: now also U5.8 (LED2)
- net HEADTILT1RPWM: now also U5.9 (LED3)
- net HEADTILT2EN: now also U1.8 (6_OUT1D)
- net HEADTILT2LPWM: now also U5.10 (LED4)
- net HEADTILT2RPWM: now also U5.11 (LED5)
- net LED1: now also U1.11 (9_OUT1C)
- net LED10: now also U1.19 (27_A13_SCK1)
- net LED2: now also U1.12 (10_CS_MQSR)
- net LED3: now also U1.42 (20_A6_TX5_LRCLK1)
- net LED4: now also U1.43 (21_A7_RX5_BCLK1)
- net LED5: now also U1.44 (22_A8_CTX1)
- net LED6: now also U1.45 (23_A9_CRX1_MCLK1)
- net LED7: now also U1.16 (24_A10_TX6_SCL2)
- net LED8: now also U1.17 (25_A11_RX6_SDA2)
- net LED9: now also U1.18 (26_A12_MOSI1)
- net MOUTHSERVO: now also U5.17 (LED10)
- net SCL: now also U1.41 (19_A5_SCL), U5.26 (SCL), U8.3 (SCL)
- net SDA: now also U1.40 (18_A4_SDA), U5.27 (SDA), U8.4 (SDA)
- net TORSOPANDIR: now also U1.5 (3_LRCLK2)
- net TORSOPANEN: now also R49.2, U1.4 (2_OUT2); no longer R49.1
- net TORSOPANPWM: now also U5.6 (LED0)
- net TORSOPANST: now also U1.6 (4_BCLK2)
- net TORSOTILT1EN: now also U1.9 (7_RX2_OUT1A)
- net TORSOTILT1LPWM: now also U5.12 (LED6)
- net TORSOTILT1RPWM: now also U5.13 (LED7)
- net TORSOTILT2EN: now also U1.10 (8_TX2_IN1)
- net TORSOTILT2LPWM: now also U5.15 (LED8)
- net TORSOTILT2RPWM: now also U5.16 (LED9)
- net VSENSE: now also U1.39 (17_A3_TX4_SDA1)
- net at R9.1: now also U5.23 (*OE)
- net at R36.2: now also U1.38 (16_A2_RX4_SCL1)
- net TORSO1 renamed TORSO
- no-connect marks 36 -> 54
Other:
- note added: "PWM Driver"
- note added: "TORSO TILT POTENTIOMETER"
- note removed: "HEAD ENCODER"
- note removed: "HEAD PAN ENCODER"
- note removed: "Shift Registers"
- note removed: "TORSO ENCODER"
- note removed: "TORSO PAN ENCODER"
- note removed: "TORSO TILT POTENTIOMETERS"
- moved on the sheet: C1, C10, C2, C3, C4, C5, C9, D1, D10, D11, D12, D13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

Commit message: Pre-flight main board
Parts:
- removed R9: 10K, Resistor10K:CRCW060310K0FKEA, symbol Device:R_US
- removed U5: PCA9685PW_118, PWMDriver:PCA9685PW,118, symbol PWMDriver:PCA9685PW_118
- added U5, U9: 74HCT125D, LevelShifter:74HCT125D, symbol LevelShifter:74HCT125D
Connections:
- net +3.3V: now also U1.46 (3V3); no longer R100.2, R101.2, R102.2, R103.2, R104.2, R105.2, R106.2, R107.2, R98.2, R99.2
- net GND: now also U10.1 (LED1-), U10.10 (LED10-), U10.2 (LED2-), U10.3 (LED3-), U10.4 (LED4-), U10.5 (LED5-), U10.6 (LED6-), U10.7 (LED7-), U10.8 (LED8-), U10.9 (LED9-), U5.1 (1OE*), U5.10 (3OE*), U5.4 (2OE*), U5.7 (GND), U9.1 (1OE*), U9.10 (3OE*), U9.4 (2OE*), U9.7 (GND)
- net HEADPANDIR: now also U5.9 (3A); no longer J10.3 (Pin_3)
- net HEADPANEN: now also U5.2 (1A); no longer J10.4 (Pin_4), R48.1
- net HEADPANPUL: now also U1.4 (2_OUT2), U5.5 (2A*); no longer R33.2
- net HEADTILT1EN: now also U1.9 (7_RX2_OUT1A); no longer U1.7 (5_IN2)
- net HEADTILT1LPWM: now also U1.11 (9_OUT1C)
- net HEADTILT1RPWM: now also U1.12 (10_CS_MQSR)
- net HEADTILT2EN: now also U1.10 (8_TX2_IN1); no longer U1.8 (6_OUT1D)
- net HEADTILT2LPWM: now also U1.13 (11_MOSI_CTX1)
- net HEADTILT2RPWM: now also U1.14 (12_MISO_MQSL)
- net LED1: now also R98.2, U1.16 (24_A10_TX6_SCL2); no longer U1.11 (9_OUT1C), U10.1 (LED1-)
- net LED10: now also R107.2, U1.27 (35_TX8); no longer U1.19 (27_A13_SCK1), U10.10 (LED10-)
- net LED2: now also R99.2, U1.17 (25_A11_RX6_SDA2); no longer U1.12 (10_CS_MQSR), U10.2 (LED2-)
- net LED3: now also R100.2, U1.18 (26_A12_MOSI1); no longer U1.42 (20_A6_TX5_LRCLK1), U10.3 (LED3-)
- net LED4: now also R101.2, U1.19 (27_A13_SCK1); no longer U1.43 (21_A7_RX5_BCLK1), U10.4 (LED4-)
- net LED5: now also R102.2, U1.22 (30_CRX3); no longer U1.44 (22_A8_CTX1), U10.5 (LED5-)
- net LED6: now also R103.2, U1.23 (31_CTX3); no longer U1.45 (23_A9_CRX1_MCLK1), U10.6 (LED6-)
- net LED7: now also R104.2, U1.24 (32_OUT1B); no longer U1.16 (24_A10_TX6_SCL2), U10.7 (LED7-)
- net LED8: now also R105.2, U1.25 (33_MCLK2); no longer U1.17 (25_A11_RX6_SDA2), U10.8 (LED8-)
- net LED9: now also R106.2, U1.26 (34_RX8); no longer U1.18 (26_A12_MOSI1), U10.9 (LED9-)
- net MOUTHSERVO: now also U1.28 (36_CS)
- net TORSOPANDIR: now also U1.6 (4_BCLK2), U9.9 (3A); no longer J11.3 (Pin_3), U1.5 (3_LRCLK2)
- net TORSOPANEN: now also U1.5 (3_LRCLK2), U9.2 (1A); no longer J11.1 (Pin_1), R49.2, U1.4 (2_OUT2)
- net TORSOPANPWM: now also U1.7 (5_IN2), U9.5 (2A*); no longer R32.2
- net TORSOTILT1EN: now also U1.42 (20_A6_TX5_LRCLK1); no longer U1.9 (7_RX2_OUT1A)
- net TORSOTILT1LPWM: now also U1.44 (22_A8_CTX1)
- net TORSOTILT1RPWM: now also U1.45 (23_A9_CRX1_MCLK1)
- net TORSOTILT2EN: now also U1.43 (21_A7_RX5_BCLK1); no longer U1.10 (8_TX2_IN1)
- net TORSOTILT2LPWM: now also U1.20 (28_RX7)
- net TORSOTILT2RPWM: now also U1.21 (29_TX7)
- net +5V: now reaches U1.49 (VUSB)
- net +5V: now also U5.13 (4OE*), U5.14 (VCC), U9.13 (4OE*), U9.14 (VCC)
- net TORSOPANST: no longer names the net of J11.7 (Pin_7)
- net TORSOPANST: no longer U1.6 (4_BCLK2)
- new net HEADPANDIR5V: J10.3 (Pin_3), U5.8 (3Y)
- new net HEADPANEN5V: J10.4 (Pin_4), R48.1, U5.3 (1Y)
- new net HEADPANPUL5V: R33.2, U5.6 (2Y)
- new net TORSOPANDIR5V: J11.3 (Pin_3), U9.8 (3Y)
- new net TORSOPANEN5V: J11.1 (Pin_1), R49.2, U9.3 (1Y)
- new net TORSOPANPWM5V: R32.2, U9.6 (2Y)
- no-connect marks 54 -> 42
Other:
- note added: "Activity Indicators (Blue)"
- note added: "Level Shifters 3.3V to 5V"
- note added: "MOUTH POSITION CONTROL SERVO"
- note added: "Motors"
- note added: "SIDE WITH PART NUMBER PRINTED"
- note added: "Servos"
- note added: "Status Indicators (Red)"
- note added: "TORSO VELOCITY CONTROL SERVO"
- note removed: "Activity Indicators"
- note removed: "Actuators"
- note removed: "MOUTH SERVO"
- note removed: "PWM Driver"
- note removed: "Status Indicators"
- note removed: "TORSO MOTOR"
- moved on the sheet: C1, C10, C2, C3, C4, C5, C9, D1, D10, D11, D12, D13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

Commit message: Re-finalize audio board and cleanup
Changed lines of the file:
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@@
 	)
 	(rectangle
-		(start 36.83 316.23)
+		(start 35.56 316.23)
 		(end 118.11 365.76)
 		(stroke
@@
 	(text "555 Timer"
 		(exclude_from_sim no)
-		(at 205.74 309.88 0)
+		(at 205.74 311.15 0)
 		(effects
 			(font
@@
 	(text "Voltage Sensing"
 		(exclude_from_sim no)
-		(at 53.34 320.04 0)
+		(at 53.34 321.31 0)
 		(effects
 			(font
@@
 	(text "Current Sensing"
 		(exclude_from_sim no)
-		(at 139.7 320.04 0)
-		(effects
-			(font
+		(at 139.7 321.31 0)
+		(effects
+			(font
