File: boards/MainRobotBoardTeensy/MainRobotBoardTeensy.kicad_sch (KiCad schematic)
At the start: 162 parts, among them J1 Screw_Terminal_01x02, J10 B4B-XH-A, J11 IDC, J2 B3B-XH-A, J3 B3B-XH-A, J5 B3B-XH-A, J6 B3B-XH-A, J7 B3B-XH-A, J8 B3B-XH-A, J9 B3B-XH-A, Q1 AO3400A, Q10 AO3400A, Q11 AO3400A, Q12 AO3400A, Q13 AO3400A, Q14 AO3400A, Q15 AO3400A, Q16 AO3400A, Q17 AO3400A, Q18 AO3400A, Q19 AO3400A, Q2 AO3400A, Q20 AO3400A, Q3 AO3400A, Q4 AO3400A, Q5 AO3400A, Q6 AO3400A, Q9 AO3400A, U1 Teensy4.1, U10 KWL-R1025BB, U11 SSD1306, U2 TLC555CDR, U3 SN74HC08DR, U4 SN74HC08DR, U5 74HCT125D, U6 SN74HC08DR, U7 ACS37220, U8 SSD1306, U9 74HCT125D

Commit message: Main robot board 5V and 7V routing
Parts:
- added J4: Screw_Terminal_01x02, TerminalBlock_Phoenix:TerminalBlock_Phoenix_MKDS-1,5-2-5.08_1x02_P5.08mm_Horizontal, symbol Connector:Screw_Terminal_01x02
Connections:
- net +3.3V: no longer J10.1 (Pin_1), J9.2 (Pin_2)
- net +5V: now also J10.1 (Pin_1); no longer U5.13 (4OE*)
- net GND: now also U5.13 (4OE*), J4.2 (Pin_2)
- net MOUTHSERVO: now also U5.12 (4A); no longer R31.2
- net MOUTHSERVO5V: now reaches U5.11 (4Y)
- net MOUTHSERVO5V: now also R31.2
- new net +7.5V: J4.1 (Pin_1), J9.2 (Pin_2)
- no-connect marks 42 -> 40
Other:
- note added: "Servo Power 7.5V"
- moved on the sheet: U5, U9
